File: Hardware/Production/Qwiic MP3-Panel.brd (EAGLE design)
At the start: 203.5 x 167.1 mm, 1662 parts, among them J1 MICRO-SD, J105 MICRO-SD, J106 ISP, J107 Poke-Home, J108 3.5mm Audio, J110 PTH, J117 MICRO-SD, J118 ISP, J119 Poke-Home, J120 3.5mm Audio, J122 PTH, J129 MICRO-SD, J130 ISP, J131 Poke-Home, J132 3.5mm Audio, J134 PTH, J14 PTH, J141 MICRO-SD, J142 ISP, J143 Poke-Home, J144 3.5mm Audio, J146 PTH, J153 MICRO-SD, J154 ISP, J155 Poke-Home, J156 3.5mm Audio, J158 PTH, J165 MICRO-SD, J166 ISP, J167 Poke-Home, J168 3.5mm Audio, J170 PTH, J177 MICRO-SD, J178 ISP, J179 Poke-Home, J180 3.5mm Audio, J182 PTH, J189 MICRO-SD, J190 ISP, J191 Poke-Home, J192 3.5mm Audio, J194 PTH, J201 MICRO-SD, J202 ISP, J203 Poke-Home, J204 3.5mm Audio, J206 PTH, J21 MICRO-SD, J213 MICRO-SD, J214 ISP, J215 Poke-Home, J216 3.5mm Audio, J22 ISP, J23 Poke-Home, J24 3.5mm Audio, J26 PTH, J3 PTH, J33 MICRO-SD, J34 ISP, J35 Poke-Home, J36 3.5mm Audio, J38 PTH, J45 MICRO-SD, J46 ISP, J47 Poke-Home, J48 3.5mm Audio, J50 PTH, J57 MICRO-SD, J58 ISP, J59 Poke-Home, J60 3.5mm Audio, J62 PTH, J69 MICRO-SD, J7 ISP, J70 ISP, J71 Poke-Home, J72 3.5mm Audio, J74 PTH, J8 3.5mm Audio, J81 MICRO-SD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

Commit message: Adding basic firmware
Parts:
- removed C100, C101, C102, C103, C106, C107, C108, C109, C110, C113, C114, C115, C116, C117, C120, C121, C122, C123, C124, C81, C82, C85, C86, C87, C88, C89, C92, C93, C94, C95, C96, C99: 0.1uF, SparkFun-Capacitors:0603
- removed C104, C111, C118, C125, C83, C90, C97: 1.0uF, SparkFun-Capacitors:0603
- removed C105, C112, C119, C126, C84, C91, C98: 1.0uF, SparkFun-Capacitors:0603-CAP
- removed D10, D11, D12, D13, D14, D15, D16, D17, D18, D9: RED, SparkFun-LED:LED-0603
- removed J100, J101, J112, J113, J124, J125, J136, J137, J148, J149, J160, J161, J172, J173, J184, J185, J196, J197, J208, J209: (no value), SparkFun-Connectors:1X01_NO_SILK
- removed J102, J114, J126, J138, J150, J162, J174, J186, J198, J210: (no value), SparkFun-Connectors:USB-MICROB-PTH-2
- removed J103, J104, J115, J116, J127, J128, J139, J140, J151, J152, J163, J164, J175, J176, J187, J188, J199, J200, J211, J212: (no value), SparkFun-Connectors:1X04_NO_SILK
- removed J105, J117, J129, J141, J153, J165, J177, J189, J201, J213: MICRO-SD, SparkFun-Connectors:MICRO-SD-SOCKET
- removed J106, J118, J130, J142, J154, J166, J178, J190, J202, J214: ISP, SparkFun-Connectors:2X3_TEST_POINTS
- removed J107, J119, J131, J143, J155, J167, J179, J191, J203, J215: Poke-Home, SparkFun-Connectors:1X02_POKEHOME
- removed J108, J120, J132, J144, J156, J168, J180, J192, J204, J216: 3.5mm Audio, SparkFun-Connectors:AUDIO_JACK_3.5MM_TRRS_SMD_RA
- removed J109, J111, J121, J123, J133, J135, J145, J147, J157, J159, J169, J171, J181, J183, J193, J195, J205, J207, J97, J99: (no value), SparkFun-Connectors:1X04_1MM_RA
- removed J110, J122, J134, J146, J158, J170, J182, J194, J206, J98: PTH, SparkX:1X04_NO_SILK
- removed JP100, JP101, JP102, JP111, JP112, JP113, JP114, JP123, JP124, JP125, JP126, JP135, JP136, JP137, JP138, JP147, JP148, JP149, JP150, JP159, JP160, JP161, JP162, JP171, JP172, JP173, JP174, JP183, JP184, JP185, JP186, JP195, JP196, JP197, JP198, JP207, JP208, JP209, JP210, JP99: FIDUCIALUFIDUCIAL, SparkFun:MICRO-FIDUCIAL
- removed JP103, JP115, JP127, JP139, JP151, JP163, JP175, JP187, JP199, JP211: Optional PTH, SparkFun-Connectors:1X03_NO_SILK
- removed JP104, JP116, JP128, JP140, JP152, JP164, JP176, JP188, JP200, JP212: PTH, SparkFun-Connectors:1X02_NO_SILK
- removed JP105, JP117, JP129, JP141, JP153, JP165, JP177, JP189, JP201, JP213: ADR, SparkFun-Jumpers:SMT-JUMPER_2_NO_NO-SILK
- removed JP106, JP118, JP130, JP142, JP154, JP166, JP178, JP190, JP202, JP214: (no value), SparkFun-Jumpers:SMT-JUMPER_3_2-NC_TRACE_SILK
- removed JP107, JP108, JP109, JP110, JP119, JP120, JP121, JP122, JP131, JP132, JP133, JP134, JP143, JP144, JP145, JP146, JP155, JP156, JP157, JP158, JP167, JP168, JP169, JP170, JP179, JP180, JP181, JP182, JP191, JP192, JP193, JP194, JP203, JP204, JP205, JP206, JP215, JP216, JP97, JP98: STAND-OFF, SparkFun:STAND-OFF
- removed LOGO10, LOGO11, LOGO12, LOGO13, LOGO14, LOGO15, LOGO16, LOGO17, LOGO18, LOGO9: OSHW-LOGOMINI, SparkFun-Aesthetics:OSHW-LOGO-MINI
- removed R100, R105, R107, R109, R110, R115, R117, R119, R120, R125, R127, R129, R130, R135, R137, R139, R140, R145, R147, R149, R150, R155, R157, R159, R160, R165, R167, R169, R170, R175, R177, R179, R180, R85, R87, R89, R90, R95, R97, R99: 10k, SparkFun-Resistors:0603
- removed R101, R111, R121, R131, R141, R151, R161, R171, R81, R91: 1k, SparkFun-Resistors:0603
- removed R102, R103, R108, R112, R113, R118, R122, R123, R128, R132, R133, R138, R142, R143, R148, R152, R153, R158, R162, R163, R168, R172, R173, R178, R82, R83, R88, R92, R93, R98: 2.2k, SparkFun-Resistors:0603
- removed R104, R106, R114, R116, R124, R126, R134, R136, R144, R146, R154, R156, R164, R166, R174, R176, R84, R86, R94, R96: 4.7k, SparkFun-Resistors:0603
- removed U$369, U$411, U$414, U$456, U$459, U$501, U$504, U$546, U$549, U$591, U$594, U$636, U$639, U$681, U$684, U$726, U$729, U$771, U$774: (no value), Labels-0_04:SDA8
- removed U$370, U$410, U$415, U$455, U$460, U$500, U$505, U$545, U$550, U$590, U$595, U$635, U$640, U$680, U$685, U$725, U$730, U$770, U$775: (no value), Labels-0_04:SCL9
- removed U$371, U$416, U$461, U$506, U$551, U$596, U$641, U$686, U$731, U$776: (no value), Labels:I_SUPER2_C-()-03
- removed U$372, U$373, U$417, U$418, U$462, U$463, U$507, U$508, U$552, U$553, U$597, U$598, U$642, U$643, U$687, U$688, U$732, U$733, U$777, U$778: (no value), Labels:INT#-[<
- removed U$374, U$375, U$419, U$420, U$464, U$465, U$509, U$510, U$554, U$555, U$599, U$600, U$644, U$645, U$689, U$690, U$734, U$735, U$779, U$780: (no value), Labels:RST#-[>
- removed U$376, U$421, U$466, U$511, U$556, U$601, U$646, U$691, U$736, U$781: (no value), Labels:PWR-()-03
- removed U$377, U$422, U$467, U$512, U$557, U$602, U$647, U$692, U$737, U$782: (no value), Labels:ADR-()-03
- removed U$378, U$402, U$423, U$447, U$468, U$492, U$513, U$537, U$558, U$582, U$603, U$627, U$648, U$672, U$693, U$717, U$738, U$762, U$783, U$807: (no value), buzzard_labels (13):TRIGGER5
- removed U$379, U$400, U$424, U$445, U$469, U$490, U$514, U$535, U$559, U$580, U$604, U$625, U$649, U$670, U$694, U$715, U$739, U$760, U$784, U$805: (no value), buzzard_labels (14):21
- removed U$380, U$396, U$425, U$441, U$470, U$486, U$515, U$531, U$560, U$576, U$605, U$621, U$650, U$666, U$695, U$711, U$740, U$756, U$785, U$801: (no value), buzzard_labels (14):32
- removed U$381, U$395, U$426, U$440, U$471, U$485, U$516, U$530, U$561, U$575, U$606, U$620, U$651, U$665, U$696, U$710, U$741, U$755, U$786, U$800: (no value), buzzard_labels (14):43
- removed U$382, U$394, U$427, U$439, U$472, U$484, U$517, U$529, U$562, U$574, U$607, U$619, U$652, U$664, U$697, U$709, U$742, U$754, U$787, U$799: (no value), buzzard_labels (16):#5
- removed U$383, U$388, U$393, U$397, U$428, U$433, U$438, U$442, U$473, U$478, U$483, U$487, U$518, U$523, U$528, U$532, U$563, U$568, U$573, U$577, U$608, U$613, U$618, U$622, U$653, U$658, U$663, U$667, U$698, U$703, U$708, U$712, U$743, U$748, U$753, U$757, U$788, U$793, U$798, U$802: (no value), buzzard_labels (16):#6
- removed U$384, U$401, U$429, U$446, U$474, U$491, U$519, U$536, U$564, U$581, U$609, U$626, U$654, U$671, U$699, U$716, U$744, U$761, U$789, U$806: (no value), buzzard_labels (16):1_1
- removed U$385, U$403, U$430, U$448, U$475, U$493, U$520, U$538, U$565, U$583, U$610, U$628, U$655, U$673, U$700, U$718, U$745, U$763, U$790, U$808: (no value), buzzard_labels (16):GND0
- removed U$386, U$399, U$431, U$444, U$476, U$489, U$521, U$534, U$566, U$579, U$611, U$624, U$656, U$669, U$701, U$714, U$746, U$759, U$791, U$804: (no value), buzzard_labels (16):L12
- removed U$387, U$398, U$432, U$443, U$477, U$488, U$522, U$533, U$567, U$578, U$612, U$623, U$657, U$668, U$702, U$713, U$747, U$758, U$792, U$803: (no value), buzzard_labels (16):R11
- removed U$389, U$404, U$434, U$449, U$479, U$494, U$524, U$539, U$569, U$584, U$614, U$629, U$659, U$674, U$704, U$719, U$749, U$764, U$794, U$809: (no value), buzzard_labels (17):PHONES0
- removed U$390, U$405, U$435, U$450, U$480, U$495, U$525, U$540, U$570, U$585, U$615, U$630, U$660, U$675, U$705, U$720, U$750, U$765, U$795, U$810: (no value), buzzard_labels (17):SPEAKER1
- removed U$391, U$392, U$436, U$437, U$481, U$482, U$526, U$527, U$571, U$572, U$616, U$617, U$661, U$662, U$706, U$707, U$751, U$752, U$796, U$797: (no value), buzzard_labels (17):QWIIC_MP32
- removed U$406, U$451, U$496, U$541, U$586, U$631, U$676, U$721, U$766: SPARKX-LOGO4, SparkX:SPARKX-MEDIUM
- removed U$407, U$452, U$497, U$542, U$587, U$632, U$677, U$722, U$767: SPARKX-LOGO3, SparkX:SPARKX-SMALL
- removed U$408, U$413, U$453, U$458, U$498, U$503, U$543, U$548, U$588, U$593, U$633, U$638, U$678, U$683, U$723, U$728, U$768, U$773: (no value), Labels-0_04:3#3V2
- removed U$409, U$412, U$454, U$457, U$499, U$502, U$544, U$547, U$589, U$592, U$634, U$637, U$679, U$682, U$724, U$727, U$769, U$772: (no value), Labels-0_04:GND1
- removed U33, U37, U41, U45, U49, U53, U57, U61, U65, U69: WT2003S, WT2003S:SO16
- removed U34, U38, U42, U46, U50, U54, U58, U62, U66, U70: TPA2005D1DRB, mike-temp:QFN-8_PAD
- removed U35, U39, U43, U47, U51, U55, U59, U63, U67, U71: ATTINY84-ARDUINO, SparkFun-IC-Microcontroller:SO14
- removed U36, U40, U44, U48, U52, U56, U60, U64, U68, U72: AP2112-3.3V, SparkFun-PowerIC:SOT23-5
- C1, C11, C18, C19, C22, C29, C3, C32, C38, C39, C52, C58, C59, C6, C68, C72, C78, C79: value 0.1uF -> 10uF
- C13, C21, C35: value 1.0uF -> 0.1uF; device SparkFun-Capacitors:0603-CAP -> SparkFun-Capacitors:0603
- C15, C23, C26, C33, C36, C4, C43, C46, C53, C66, C73: value 0.1uF -> 1.0uF
- C17, C30, C37, C40, C47, C50, C57, C60, C67, C80, C9: value 0.1uF -> 1.0uF; device SparkFun-Capacitors:0603 -> SparkFun-Capacitors:0603-CAP
- C20, C27: device SparkFun-Capacitors:0603 -> SparkFun-Capacitors:0603-CAP
- C28, C42, C49: value 1.0uF -> 10uF; device SparkFun-Capacitors:0603-CAP -> SparkFun-Capacitors:0603
- C34, C41, C55: value 1.0uF -> 0.1uF
- C48, C62, C69: value 1.0uF -> 10uF
- C56, C63: device SparkFun-Capacitors:0603-CAP -> SparkFun-Capacitors:0603
- J18, J30, J42, J54, J6, J66, J78, J90: device SparkFun-Connectors:USB-MICROB-PTH-2 -> SparkFun-Connectors:USB-MICROB-PTH-MILL
- JP10, JP19, JP31, JP43, JP55, JP67, JP79, JP91: value Optional PTH -> PTH
- R11, R16, R26, R36, R46, R56, R66, R76: value 4.7k -> 100k
- U$100, U$325, U$95: device Labels-0_04:SCL9 -> Labels-0_04:3#3V2
- U$101, U$236: device Labels:I_SUPER2_C-()-03 -> Labels-0_04:SDA8
- U$102, U$148, U$327: device Labels:INT#-[< -> Labels-0_04:SCL9
- U$103, U$57: device Labels:INT#-[< -> Labels:I_SUPER2_C-()-03
- U$104, U$105, U$150, U$59: device Labels:RST#-[> -> Labels:INT#-[<
- U$106, U$61: device Labels:PWR-()-03 -> Labels:RST#-[>
- U$107, U$152: device Labels:ADR-()-03 -> Labels:RST#-[>
- U$108: device buzzard_labels (13):TRIGGER5 -> Labels:PWR-()-03
- U$109: device buzzard_labels (14):21 -> Labels:ADR-()-03
- U$110: device buzzard_labels (14):32 -> buzzard_labels (13):TRIGGER5
- U$111: device buzzard_labels (14):43 -> buzzard_labels (14):21
- U$112: device buzzard_labels (16):#5 -> buzzard_labels (14):32
- U$113, U$127, U$343: device buzzard_labels (16):#6 -> buzzard_labels (14):43
- U$114, U$356: device buzzard_labels (16):1_1 -> buzzard_labels (16):#5
- U$115, U$313: device buzzard_labels (16):GND0 -> buzzard_labels (16):#6
- U$116: device buzzard_labels (16):L12 -> buzzard_labels (16):1_1
- U$117: device buzzard_labels (16):R11 -> buzzard_labels (16):GND0
- U$118, U$348: device buzzard_labels (16):#6 -> buzzard_labels (16):L12
- U$119, U$314: device buzzard_labels (17):PHONES0 -> buzzard_labels (16):R11
- U$120, U$345: device buzzard_labels (17):SPEAKER1 -> buzzard_labels (16):#6
- U$121, U$167: device buzzard_labels (17):QWIIC_MP32 -> buzzard_labels (17):PHONES0
- U$122, U$76: device buzzard_labels (17):QWIIC_MP32 -> buzzard_labels (17):SPEAKER1
- U$123, U$262, U$307, U$78: device buzzard_labels (16):#6 -> buzzard_labels (17):QWIIC_MP32
- U$124, U$169: device buzzard_labels (16):#5 -> buzzard_labels (17):QWIIC_MP32
- U$125, U$350: device buzzard_labels (14):43 -> buzzard_labels (16):#6
- U$126: device buzzard_labels (14):32 -> buzzard_labels (16):#5
- U$128, U$342: device buzzard_labels (16):R11 -> buzzard_labels (14):32
- U$129, U$161, U$309: device buzzard_labels (16):L12 -> buzzard_labels (16):#6
- U$130: device buzzard_labels (14):21 -> buzzard_labels (16):R11
- U$131: device buzzard_labels (16):1_1 -> buzzard_labels (16):L12
- U$132: device buzzard_labels (13):TRIGGER5 -> buzzard_labels (14):21
- U$133, U$70: device buzzard_labels (16):GND0 -> buzzard_labels (16):1_1
- U$134: device buzzard_labels (17):PHONES0 -> buzzard_labels (13):TRIGGER5
- U$135, U$255: device buzzard_labels (17):SPEAKER1 -> buzzard_labels (16):GND0
- U$136: value SPARKX-LOGO4 -> (none); device SparkX:SPARKX-MEDIUM -> buzzard_labels (17):PHONES0
- U$137: value SPARKX-LOGO3 -> (none); device SparkX:SPARKX-SMALL -> buzzard_labels (17):SPEAKER1
- U$138, U$368: device Labels-0_04:3#3V2 -> Labels:QWIIC-LOGO-MEDIUM
- U$139, U$277: value (none) -> SPARKX-LOGO4; device Labels-0_04:GND1 -> SparkX:SPARKX-MEDIUM
- U$140: value (none) -> SPARKX-LOGO3; device Labels-0_04:SCL9 -> SparkX:SPARKX-SMALL
- U$141, U$279, U$54: device Labels-0_04:SDA8 -> Labels-0_04:3#3V2
- U$143: device Labels-0_04:3#3V2 -> Labels-0_04:SCL9
- U$145, U$280, U$50: device Labels-0_04:SCL9 -> Labels-0_04:GND1
- U$146: device Labels:I_SUPER2_C-()-03 -> Labels-0_04:3#3V2
- U$147, U$193, U$282, U$328: device Labels:INT#-[< -> Labels-0_04:SDA8
- U$149, U$195: device Labels:RST#-[> -> Labels:I_SUPER2_C-()-03
- U$151, U$196: device Labels:PWR-()-03 -> Labels:INT#-[<
- U$153, U$198: device buzzard_labels (13):TRIGGER5 -> Labels:RST#-[>
- U$154: device buzzard_labels (14):21 -> Labels:PWR-()-03
- U$155: device buzzard_labels (14):32 -> Labels:ADR-()-03
- U$156: device buzzard_labels (14):43 -> buzzard_labels (13):TRIGGER5
- U$157: device buzzard_labels (16):#5 -> buzzard_labels (14):21
- U$158, U$82: device buzzard_labels (16):#6 -> buzzard_labels (14):32
- U$159, U$311: device buzzard_labels (16):1_1 -> buzzard_labels (14):43
- U$160: device buzzard_labels (16):GND0 -> buzzard_labels (16):#5
- U$162: device buzzard_labels (16):R11 -> buzzard_labels (16):1_1
- U$163: device buzzard_labels (16):#6 -> buzzard_labels (16):GND0
- U$164, U$269: device buzzard_labels (17):PHONES0 -> buzzard_labels (16):L12
- U$165, U$360: device buzzard_labels (17):SPEAKER1 -> buzzard_labels (16):R11
- U$166, U$212: device buzzard_labels (17):QWIIC_MP32 -> buzzard_labels (16):#6
- U$168, U$352: device buzzard_labels (16):#6 -> buzzard_labels (17):SPEAKER1
- U$170, U$215: device buzzard_labels (14):43 -> buzzard_labels (17):QWIIC_MP32
- U$171: device buzzard_labels (14):32 -> buzzard_labels (16):#6
- U$172, U$298, U$68: device buzzard_labels (16):#6 -> buzzard_labels (16):#5
- U$173, U$297: device buzzard_labels (16):R11 -> buzzard_labels (14):43
- U$174, U$296: device buzzard_labels (16):L12 -> buzzard_labels (14):32
- U$175, U$355: device buzzard_labels (14):21 -> buzzard_labels (16):#6
- U$176: device buzzard_labels (16):1_1 -> buzzard_labels (16):R11
- U$177: device buzzard_labels (13):TRIGGER5 -> buzzard_labels (16):L12
- U$178, U$295: device buzzard_labels (16):GND0 -> buzzard_labels (14):21
- U$179, U$254: device buzzard_labels (17):PHONES0 -> buzzard_labels (16):1_1
- U$180: device buzzard_labels (17):SPEAKER1 -> buzzard_labels (13):TRIGGER5
- U$181: value SPARKX-LOGO4 -> (none); device SparkX:SPARKX-MEDIUM -> buzzard_labels (16):GND0
- U$182: value SPARKX-LOGO3 -> (none); device SparkX:SPARKX-SMALL -> buzzard_labels (17):PHONES0
- U$183: device Labels-0_04:3#3V2 -> buzzard_labels (17):SPEAKER1
- U$184, U$322: device Labels-0_04:GND1 -> Labels:QWIIC-LOGO-MEDIUM
- U$185: value (none) -> SPARKX-LOGO4; device Labels-0_04:SCL9 -> SparkX:SPARKX-MEDIUM
- U$186, U$324: value (none) -> SPARKX-LOGO3; device Labels-0_04:SDA8 -> SparkX:SPARKX-SMALL
- U$187, U$49: device Labels-0_04:GND1 -> Labels-0_04:3#3V2
- U$188, U$53: device Labels-0_04:3#3V2 -> Labels-0_04:GND1
- U$189, U$51: device Labels-0_04:SDA8 -> Labels-0_04:SCL9
- U$190, U$55: device Labels-0_04:SCL9 -> Labels-0_04:SDA8
- U$191, U$326: device Labels:I_SUPER2_C-()-03 -> Labels-0_04:GND1
- U$192, U$238: device Labels:INT#-[< -> Labels-0_04:3#3V2
- U$194, U$240: device Labels:RST#-[> -> Labels-0_04:SCL9
- U$197, U$242: device Labels:ADR-()-03 -> Labels:INT#-[<
- U$199, U$244: device buzzard_labels (14):21 -> Labels:RST#-[>
- U$200: device buzzard_labels (14):32 -> Labels:PWR-()-03
- U$201: device buzzard_labels (14):43 -> Labels:ADR-()-03
- U$202: device buzzard_labels (16):#5 -> buzzard_labels (13):TRIGGER5
- U$203: device buzzard_labels (16):#6 -> buzzard_labels (14):21
- U$204, U$266: device buzzard_labels (16):1_1 -> buzzard_labels (14):32
- U$205: device buzzard_labels (16):GND0 -> buzzard_labels (14):43
- U$206, U$264: device buzzard_labels (16):L12 -> buzzard_labels (16):#5
- U$207, U$263, U$83: device buzzard_labels (16):R11 -> buzzard_labels (16):#6
- U$208: device buzzard_labels (16):#6 -> buzzard_labels (16):1_1
- U$209, U$89: device buzzard_labels (17):PHONES0 -> buzzard_labels (16):GND0
- U$210, U$315: device buzzard_labels (17):SPEAKER1 -> buzzard_labels (16):L12
- U$211, U$257: device buzzard_labels (17):QWIIC_MP32 -> buzzard_labels (16):R11
- U$213: device buzzard_labels (16):#6 -> buzzard_labels (17):PHONES0
- U$214: device buzzard_labels (16):#5 -> buzzard_labels (17):SPEAKER1
- U$216, U$261: device buzzard_labels (14):32 -> buzzard_labels (17):QWIIC_MP32
- U$218, U$252: device buzzard_labels (16):R11 -> buzzard_labels (16):#5
- U$219, U$251: device buzzard_labels (16):L12 -> buzzard_labels (14):43
- U$220: device buzzard_labels (14):21 -> buzzard_labels (14):32
- U$221, U$69: device buzzard_labels (16):1_1 -> buzzard_labels (16):#6
- U$222: device buzzard_labels (13):TRIGGER5 -> buzzard_labels (16):R11
- U$223: device buzzard_labels (16):GND0 -> buzzard_labels (16):L12
- U$224: device buzzard_labels (17):PHONES0 -> buzzard_labels (14):21
- U$225, U$300: device buzzard_labels (17):SPEAKER1 -> buzzard_labels (16):1_1
- U$226: value SPARKX-LOGO4 -> (none); device SparkX:SPARKX-MEDIUM -> buzzard_labels (13):TRIGGER5
- U$227: value SPARKX-LOGO3 -> (none); device SparkX:SPARKX-SMALL -> buzzard_labels (16):GND0
- U$228: device Labels-0_04:3#3V2 -> buzzard_labels (17):PHONES0
- U$229, U$367: device Labels-0_04:GND1 -> buzzard_labels (17):SPEAKER1
- U$230: device Labels-0_04:SCL9 -> Labels:QWIIC-LOGO-MEDIUM
- U$231: value (none) -> SPARKX-LOGO4; device Labels-0_04:SDA8 -> SparkX:SPARKX-MEDIUM
- U$232, U$94: value (none) -> SPARKX-LOGO3; device Labels-0_04:GND1 -> SparkX:SPARKX-SMALL
- U$234, U$96, U$99: device Labels-0_04:SDA8 -> Labels-0_04:GND1
- U$237, U$283: device Labels:INT#-[< -> Labels-0_04:GND1
- U$239, U$285: device Labels:RST#-[> -> Labels-0_04:SDA8
- U$241: device Labels:PWR-()-03 -> Labels:I_SUPER2_C-()-03
- U$243, U$288: device buzzard_labels (13):TRIGGER5 -> Labels:INT#-[<
- U$245, U$290: device buzzard_labels (14):32 -> Labels:RST#-[>
- U$246: device buzzard_labels (14):43 -> Labels:PWR-()-03
- U$247: device buzzard_labels (16):#5 -> Labels:ADR-()-03
- U$248: device buzzard_labels (16):#6 -> buzzard_labels (13):TRIGGER5
- U$249, U$86: device buzzard_labels (16):1_1 -> buzzard_labels (14):21
- U$250, U$358: device buzzard_labels (16):GND0 -> buzzard_labels (14):32
- U$256, U$302: device buzzard_labels (17):QWIIC_MP32 -> buzzard_labels (16):L12
- U$259: device buzzard_labels (16):#5 -> buzzard_labels (17):PHONES0
- U$260: device buzzard_labels (14):43 -> buzzard_labels (17):SPEAKER1
- U$265: device buzzard_labels (14):21 -> buzzard_labels (14):43
- U$267: device buzzard_labels (13):TRIGGER5 -> buzzard_labels (16):#6
- U$268: device buzzard_labels (16):GND0 -> buzzard_labels (16):R11
- U$270: device buzzard_labels (17):SPEAKER1 -> buzzard_labels (14):21
- U$271: value SPARKX-LOGO4 -> (none); device SparkX:SPARKX-MEDIUM -> buzzard_labels (16):1_1
- U$272: value SPARKX-LOGO3 -> (none); device SparkX:SPARKX-SMALL -> buzzard_labels (13):TRIGGER5
- U$273: device Labels-0_04:3#3V2 -> buzzard_labels (16):GND0
- U$274: device Labels-0_04:GND1 -> buzzard_labels (17):PHONES0
- U$275: device Labels-0_04:SCL9 -> buzzard_labels (17):SPEAKER1
- U$276: device Labels-0_04:SDA8 -> Labels:QWIIC-LOGO-MEDIUM
- U$278, U$48: value (none) -> SPARKX-LOGO3; device Labels-0_04:3#3V2 -> SparkX:SPARKX-SMALL
- U$281, U$56: device Labels:I_SUPER2_C-()-03 -> Labels-0_04:SCL9
- U$284, U$330: device Labels:RST#-[> -> Labels-0_04:3#3V2
- U$286: device Labels:PWR-()-03 -> Labels-0_04:SCL9
- U$287: device Labels:ADR-()-03 -> Labels:I_SUPER2_C-()-03
- U$289, U$334: device buzzard_labels (14):21 -> Labels:INT#-[<
- U$291, U$336: device buzzard_labels (14):43 -> Labels:RST#-[>
- U$292: device buzzard_labels (16):#5 -> Labels:PWR-()-03
- U$293: device buzzard_labels (16):#6 -> Labels:ADR-()-03
- U$294: device buzzard_labels (16):1_1 -> buzzard_labels (13):TRIGGER5
- U$299, U$359, U$74: device buzzard_labels (17):PHONES0 -> buzzard_labels (16):#6
- U$301, U$347: device buzzard_labels (17):QWIIC_MP32 -> buzzard_labels (16):GND0
- U$303, U$73: device buzzard_labels (16):#6 -> buzzard_labels (16):R11
- U$304, U$79: device buzzard_labels (16):#5 -> buzzard_labels (16):#6
- U$305: device buzzard_labels (14):43 -> buzzard_labels (17):PHONES0
- U$306: device buzzard_labels (14):32 -> buzzard_labels (17):SPEAKER1
- U$308, U$353: device buzzard_labels (16):R11 -> buzzard_labels (17):QWIIC_MP32
- U$310: device buzzard_labels (14):21 -> buzzard_labels (16):#5
- U$312: device buzzard_labels (13):TRIGGER5 -> buzzard_labels (14):32
- U$316: value SPARKX-LOGO4 -> (none); device SparkX:SPARKX-MEDIUM -> buzzard_labels (14):21
- U$317: value SPARKX-LOGO3 -> (none); device SparkX:SPARKX-SMALL -> buzzard_labels (16):1_1
- U$318: device Labels-0_04:3#3V2 -> buzzard_labels (13):TRIGGER5
- U$319: device Labels-0_04:GND1 -> buzzard_labels (16):GND0
- U$320: device Labels-0_04:SCL9 -> buzzard_labels (17):PHONES0
- U$321: device Labels-0_04:SDA8 -> buzzard_labels (17):SPEAKER1
- U$323, U$93: value (none) -> SPARKX-LOGO4; device Labels-0_04:3#3V2 -> SparkX:SPARKX-MEDIUM
- U$329: device Labels:RST#-[> -> Labels-0_04:GND1
- U$331: device Labels:PWR-()-03 -> Labels-0_04:SDA8
- U$332: device Labels:ADR-()-03 -> Labels-0_04:SCL9
- U$333: device buzzard_labels (13):TRIGGER5 -> Labels:I_SUPER2_C-()-03
- U$335: device buzzard_labels (14):32 -> Labels:INT#-[<
- U$337: device buzzard_labels (16):#5 -> Labels:RST#-[>
- U$338: device buzzard_labels (16):#6 -> Labels:PWR-()-03
- U$339: device buzzard_labels (16):1_1 -> Labels:ADR-()-03
- U$340, U$88: device buzzard_labels (16):GND0 -> buzzard_labels (13):TRIGGER5
- U$341: device buzzard_labels (16):L12 -> buzzard_labels (14):21
- U$344: device buzzard_labels (17):PHONES0 -> buzzard_labels (16):#5
- U$346: device buzzard_labels (17):QWIIC_MP32 -> buzzard_labels (16):1_1
- U$349: device buzzard_labels (16):#5 -> buzzard_labels (16):R11
- U$351: device buzzard_labels (14):32 -> buzzard_labels (17):PHONES0
- U$354: device buzzard_labels (16):L12 -> buzzard_labels (17):QWIIC_MP32
- U$357: device buzzard_labels (13):TRIGGER5 -> buzzard_labels (14):43
- U$361: value SPARKX-LOGO4 -> (none); device SparkX:SPARKX-MEDIUM -> buzzard_labels (16):L12
- U$362: value SPARKX-LOGO3 -> (none); device SparkX:SPARKX-SMALL -> buzzard_labels (14):21
- U$363: device Labels-0_04:3#3V2 -> buzzard_labels (16):1_1
- U$364: device Labels-0_04:GND1 -> buzzard_labels (13):TRIGGER5
- U$365: device Labels-0_04:SCL9 -> buzzard_labels (16):GND0
- U$366: device Labels-0_04:SDA8 -> buzzard_labels (17):PHONES0
- U$47, U$92: value SPARKX-LOGO3 -> (none); device SparkX:SPARKX-SMALL -> Labels:QWIIC-LOGO-MEDIUM
- U$52: device Labels-0_04:GND1 -> Labels-0_04:SDA8
- U$62: device Labels:ADR-()-03 -> Labels:PWR-()-03
- U$63: device buzzard_labels (13):TRIGGER5 -> Labels:ADR-()-03
- U$64: device buzzard_labels (14):21 -> buzzard_labels (13):TRIGGER5
- U$65: device buzzard_labels (14):32 -> buzzard_labels (14):21
- U$66: device buzzard_labels (14):43 -> buzzard_labels (14):32
- U$67: device buzzard_labels (16):#5 -> buzzard_labels (14):43
- U$71: device buzzard_labels (16):L12 -> buzzard_labels (16):GND0
- U$72: device buzzard_labels (16):R11 -> buzzard_labels (16):L12
- U$75, U$90: device buzzard_labels (17):SPEAKER1 -> buzzard_labels (17):PHONES0
- U$80: device buzzard_labels (14):43 -> buzzard_labels (16):#5
- U$81: device buzzard_labels (14):32 -> buzzard_labels (14):43
- U$84: device buzzard_labels (16):L12 -> buzzard_labels (16):R11
- U$85: device buzzard_labels (14):21 -> buzzard_labels (16):L12
- U$87: device buzzard_labels (13):TRIGGER5 -> buzzard_labels (16):1_1
- U$91: value SPARKX-LOGO4 -> (none); device SparkX:SPARKX-MEDIUM -> buzzard_labels (17):SPEAKER1
- U$97: device Labels-0_04:GND1 -> Labels-0_04:SCL9
- U$98: device Labels-0_04:3#3V2 -> Labels-0_04:SDA8
- U1, U10, U14, U18, U22, U26, U30, U6: value TPA2005D1DRB -> TPA2005D1; device mike-temp:QFN-8_PAD -> SparkFun-IC-Amplifiers:QFN-8_PAD
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Connections:
- removed net !INT10: J124.1, U43.6
- removed net !INT11: J136.1, U47.6
- removed net !INT12: J148.1, U51.6
- removed net !INT13: J160.1, U55.6
- removed net !INT14: J172.1, U59.6
- removed net !INT15: J184.1, U63.6
- removed net !INT16: J196.1, U67.6
- removed net !INT17: J208.1, U71.6
- removed net !INT8: J100.1, U35.6
- removed net !INT9: J112.1, U39.6
- removed net !RST10: J125.1, J130.5, R104.1, U43.4
- removed net !RST11: J137.1, J142.5, R114.1, U47.4
- removed net !RST12: J149.1, J154.5, R124.1, U51.4
- removed net !RST13: J161.1, J166.5, R134.1, U55.4
- removed net !RST14: J173.1, J178.5, R144.1, U59.4
- removed net !RST15: J185.1, J190.5, R154.1, U63.4
- removed net !RST16: J197.1, J202.5, R164.1, U67.4
- removed net !RST17: J209.1, J214.5, R174.1, U71.4
- removed net !RST8: J101.1, J106.5, R84.1, U35.4
- removed net !RST9: J113.1, J118.5, R94.1, U39.4
- removed net !SDN10: R105.1, U41.7, U42.1
- removed net !SDN11: R115.1, U45.7, U46.1
- removed net !SDN12: R125.1, U49.7, U50.1
- removed net !SDN13: R135.1, U53.7, U54.1
- removed net !SDN14: R145.1, U57.7, U58.1
- removed net !SDN15: R155.1, U61.7, U62.1
- removed net !SDN16: R165.1, U65.7, U66.1
- removed net !SDN17: R175.1, U69.7, U70.1
- removed net !SDN8: R85.1, U33.7, U34.1
- removed net !SDN9: R95.1, U37.7, U38.1
- removed net 3.3V10: C71.1, C77.1, J121.2, J122.2, J123.2, J130.2, JP130.2, R101.2, R104.2, R105.2, U42.6, U43.1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
- removed net 3.3V11: C78.1, C84.1, J133.2, J134.2, J135.2, J142.2, JP142.2, R111.2, R114.2, R115.2, U46.6, U47.1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
- removed net 3.3V12: C85.1, C91.1, J145.2, J146.2, J147.2, J154.2, JP154.2, R121.2, R124.2, R125.2, U50.6, U51.1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
- removed net 3.3V13: C92.1, C98.1, J157.2, J158.2, J159.2, J166.2, JP166.2, R131.2, R134.2, R135.2, U54.6, U55.1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
- removed net 3.3V14: C105.1, C99.1, J169.2, J170.2, J171.2, J178.2, JP178.2, R141.2, R144.2, R145.2, U58.6, U59.1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
- removed net 3.3V15: C106.1, C112.1, J181.2, J182.2, J183.2, J190.2, JP190.2, R151.2, R154.2, R155.2, U62.6, U63.1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
- removed net 3.3V16: C113.1, C119.1, J193.2, J194.2, J195.2, J202.2, JP202.2, R161.2, R164.2, R165.2, U66.6, U67.1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
- removed net 3.3V17: C120.1, C126.1, J205.2, J206.2, J207.2, J214.2, JP214.2, R171.2, R174.2, R175.2, U70.6, U71.1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
- removed net 3.3V8: C57.1, C63.1, J106.2, J97.2, J98.2, J99.2, JP106.2, R81.2, R84.2, R85.2, U34.6, U35.1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
- removed net 3.3V9: C64.1, C70.1, J109.2, J110.2, J111.2, J118.2, JP118.2, R91.2, R94.2, R95.2, U38.6, U39.1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
- removed net 5V10: C73.1, J126.VBUS, U41.5, U44.1, U44.3
- removed net 5V11: C80.1, J138.VBUS, U45.5, U48.1, U48.3
- removed net 5V12: C87.1, J150.VBUS, U49.5, U52.1, U52.3
- removed net 5V13: C94.1, J162.VBUS, U53.5, U56.1, U56.3
- removed net 5V14: C101.1, J174.VBUS, U57.5, U60.1, U60.3
- removed net 5V15: C108.1, J186.VBUS, U61.5, U64.1, U64.3
- removed net 5V16: C115.1, J198.VBUS, U65.5, U68.1, U68.3
- removed net 5V17: C122.1, J210.VBUS, U69.5, U72.1, U72.3
- removed net 5V8: C59.1, J102.VBUS, U33.5, U36.1, U36.3
- removed net 5V9: C66.1, J114.VBUS, U37.5, U40.1, U40.3
- removed net ADKEY10: R107.1, U41.13
- removed net ADKEY11: R117.1, U45.13
- removed net ADKEY12: R127.1, U49.13
- removed net ADKEY13: R137.1, U53.13
- removed net ADKEY14: R147.1, U57.13
- removed net ADKEY15: R157.1, U61.13
- removed net ADKEY16: R167.1, U65.13
- removed net ADKEY17: R177.1, U69.13
- removed net ADKEY8: R87.1, U33.13
- removed net ADKEY9: R97.1, U37.13
- removed net ADR10: JP129.2, U43.3
- removed net ADR11: JP141.2, U47.3
- removed net ADR12: JP153.2, U51.3
- removed net ADR13: JP165.2, U55.3
- removed net ADR14: JP177.2, U59.3
- removed net ADR15: JP189.2, U63.3
- removed net ADR16: JP201.2, U67.3
- removed net ADR17: JP213.2, U71.3
- removed net ADR8: JP105.2, U35.3
- removed net ADR9: JP117.2, U39.3
- removed net D+10: J126.D+, U41.12
- removed net D+11: J138.D+, U45.12
- removed net D+12: J150.D+, U49.12
- removed net D+13: J162.D+, U53.12
- removed net D+14: J174.D+, U57.12
- removed net D+15: J186.D+, U61.12
- removed net D+16: J198.D+, U65.12
- removed net D+17: J210.D+, U69.12
- removed net D+8: J102.D+, U33.12
- removed net D+9: J114.D+, U37.12
- removed net D-10: J126.D-, U41.11
- removed net D-11: J138.D-, U45.11
- removed net D-12: J150.D-, U49.11
- removed net D-13: J162.D-, U53.11
- removed net D-14: J174.D-, U57.11
- removed net D-15: J186.D-, U61.11
- removed net D-16: J198.D-, U65.11
- removed net D-17: J210.D-, U69.11
- removed net D-8: J102.D-, U33.11
- removed net D-9: J114.D-, U37.11
- removed net GND10: C71.2, C72.2, C73.2, C76.1, C77.2, D11.C, J121.1, J122.1, J123.1, J126.GND, J126.SHIELD, J126.SHIELD10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
- removed net GND11: C78.2, C79.2, C80.2, C83.1, C84.2, D12.C, J133.1, J134.1, J135.1, J138.GND, J138.SHIELD, J138.SHIELD10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
- removed net GND12: C85.2, C86.2, C87.2, C90.1, C91.2, D13.C, J145.1, J146.1, J147.1, J150.GND, J150.SHIELD, J150.SHIELD10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
- removed net GND13: C92.2, C93.2, C94.2, C97.1, C98.2, D14.C, J157.1, J158.1, J159.1, J162.GND, J162.SHIELD, J162.SHIELD10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
- removed net GND14: C100.2, C101.2, C104.1, C105.2, C99.2, D15.C, J169.1, J170.1, J171.1, J174.GND, J174.SHIELD, J174.SHIELD10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
- removed net GND15: C106.2, C107.2, C108.2, C111.1, C112.2, D16.C, J181.1, J182.1, J183.1, J186.GND, J186.SHIELD, J186.SHIELD10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
- removed net GND16: C113.2, C114.2, C115.2, C118.1, C119.2, D17.C, J193.1, J194.1, J195.1, J198.GND, J198.SHIELD, J198.SHIELD10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
- removed net GND17: C120.2, C121.2, C122.2, C125.1, C126.2, D18.C, J205.1, J206.1, J207.1, J210.GND, J210.SHIELD, J210.SHIELD10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
- removed net GND8: C57.2, C58.2, C59.2, C62.1, C63.2, D9.C, J102.GND, J102.SHIELD, J102.SHIELD10, J102.SHIELD2, J102.SHIELD3, J102.SHIELD4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
- removed net GND9: C64.2, C65.2, C66.2, C69.1, C70.2, D10.C, J109.1, J110.1, J111.1, J114.GND, J114.SHIELD, J114.SHIELD10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
- removed net IN+AMP10: R106.2, U42.3
- removed net IN+AMP11: R116.2, U46.3
- removed net IN+AMP12: R126.2, U50.3
- removed net IN+AMP13: R136.2, U54.3
- removed net IN+AMP14: R146.2, U58.3
- removed net IN+AMP15: R156.2, U62.3
- removed net IN+AMP16: R166.2, U66.3
- removed net IN+AMP17: R176.2, U70.3
- removed net IN+AMP8: R86.2, U34.3
- removed net IN+AMP9: R96.2, U38.3
- removed net IN-AMP10: R109.2, R110.2, U42.4
- removed net IN-AMP11: R119.2, R120.2, U46.4
- removed net IN-AMP12: R129.2, R130.2, U50.4
- removed net IN-AMP13: R139.2, R140.2, U54.4
- removed net IN-AMP14: R149.2, R150.2, U58.4
- removed net IN-AMP15: R159.2, R160.2, U62.4
- removed net IN-AMP16: R169.2, R170.2, U66.4
- removed net IN-AMP17: R179.2, R180.2, U70.4
- removed net IN-AMP8: R89.2, R90.2, U34.4
- removed net IN-AMP9: R100.2, R99.2, U38.4
- removed net MP3-RXI10: U41.15, U43.13
- removed net MP3-RXI11: U45.15, U47.13
- removed net MP3-RXI12: U49.15, U51.13
- removed net MP3-RXI13: U53.15, U55.13
- removed net MP3-RXI14: U57.15, U59.13
- removed net MP3-RXI15: U61.15, U63.13
- removed net MP3-RXI16: U65.15, U67.13
- removed net MP3-RXI17: U69.15, U71.13
- removed net MP3-RXI8: U33.15, U35.13
- removed net MP3-RXI9: U37.15, U39.13
- removed net MP3-TXO10: U41.16, U43.12
- removed net MP3-TXO11: U45.16, U47.12
- removed net MP3-TXO12: U49.16, U51.12
- removed net MP3-TXO13: U53.16, U55.12
- removed net MP3-TXO14: U57.16, U59.12
- removed net MP3-TXO15: U61.16, U63.12
- removed net MP3-TXO16: U65.16, U67.12
- removed net MP3-TXO17: U69.16, U71.12
- removed net MP3-TXO8: U33.16, U35.12
- removed net MP3-TXO9: U37.16, U39.12
- removed net N$33: D9.A, R81.1
- removed net N$34: C62.2, R86.1
- removed net N$35: C60.2, R89.1
- removed net N$36: C61.2, R90.1
- removed net N$37: D10.A, R91.1
- removed net N$38: C69.2, R96.1
- removed net N$39: C67.2, R99.1
- removed net N$40: C68.2, R100.1
- removed net N$41: D11.A, R101.1
- removed net N$42: C76.2, R106.1
- removed net N$43: C74.2, R109.1
- removed net N$44: C75.2, R110.1
- removed net N$45: D12.A, R111.1
- removed net N$46: C83.2, R116.1
- removed net N$47: C81.2, R119.1
- removed net N$48: C82.2, R120.1
- removed net N$49: D13.A, R121.1
- removed net N$50: C90.2, R126.1
- removed net N$51: C88.2, R129.1
- removed net N$52: C89.2, R130.1
- removed net N$53: D14.A, R131.1
- removed net N$54: C97.2, R136.1
- removed net N$55: C95.2, R139.1
- removed net N$56: C96.2, R140.1
- removed net N$57: D15.A, R141.1
- removed net N$58: C104.2, R146.1
- removed net N$59: C102.2, R149.1
- removed net N$60: C103.2, R150.1
- removed net N$61: D16.A, R151.1
- removed net N$62: C111.2, R156.1
- removed net N$63: C109.2, R159.1
- removed net N$64: C110.2, R160.1
- removed net N$65: D17.A, R161.1
- removed net N$66: C118.2, R166.1
- removed net N$67: C116.2, R169.1
- removed net N$68: C117.2, R170.1
- removed net N$69: D18.A, R171.1
- removed net N$70: C125.2, R176.1
- removed net N$71: C123.2, R179.1
- removed net N$72: C124.2, R180.1
- removed net OUT+10: J131.P1, J131.P3, JP128.1, U42.5
- removed net OUT+11: J143.P1, J143.P3, JP140.1, U46.5
- removed net OUT+12: J155.P1, J155.P3, JP152.1, U50.5
- removed net OUT+13: J167.P1, J167.P3, JP164.1, U54.5
- removed net OUT+14: J179.P1, J179.P3, JP176.1, U58.5
- removed net OUT+15: J191.P1, J191.P3, JP188.1, U62.5
- removed net OUT+16: J203.P1, J203.P3, JP200.1, U66.5
- removed net OUT+17: J215.P1, J215.P3, JP212.1, U70.5
- removed net OUT+8: J107.P1, J107.P3, JP104.1, U34.5
- removed net OUT+9: J119.P1, J119.P3, JP116.1, U38.5
- removed net OUT-10: J131.P2, J131.P4, JP128.2, U42.8
- removed net OUT-11: J143.P2, J143.P4, JP140.2, U46.8
- removed net OUT-12: J155.P2, J155.P4, JP152.2, U50.8
- removed net OUT-13: J167.P2, J167.P4, JP164.2, U54.8
- removed net OUT-14: J179.P2, J179.P4, JP176.2, U58.8
- removed net OUT-15: J191.P2, J191.P4, JP188.2, U62.8
- removed net OUT-16: J203.P2, J203.P4, JP200.2, U66.8
- removed net OUT-17: J215.P2, J215.P4, JP212.2, U70.8
- removed net OUT-8: J107.P2, J107.P4, JP104.2, U34.8
- removed net OUT-9: J119.P2, J119.P4, JP116.2, U38.8
- removed net PLAYING10: U41.14, U43.11
- removed net PLAYING11: U45.14, U47.11
- removed net PLAYING12: U49.14, U51.11
- removed net PLAYING13: U53.14, U55.11
- removed net PLAYING14: U57.14, U59.11
- removed net PLAYING15: U61.14, U63.11
- removed net PLAYING16: U65.14, U67.11
- removed net PLAYING17: U69.14, U71.11
- removed net PLAYING8: U33.14, U35.11
- removed net PLAYING9: U37.14, U39.11
- removed net SCL10: J121.4, J122.4, J123.4, J130.3, R102.1, U43.9
- removed net SCL11: J133.4, J134.4, J135.4, J142.3, R112.1, U47.9
- removed net SCL12: J145.4, J146.4, J147.4, J154.3, R122.1, U51.9
- removed net SCL13: J157.4, J158.4, J159.4, J166.3, R132.1, U55.9
- removed net SCL14: J169.4, J170.4, J171.4, J178.3, R142.1, U59.9
- removed net SCL15: J181.4, J182.4, J183.4, J190.3, R152.1, U63.9
- removed net SCL16: J193.4, J194.4, J195.4, J202.3, R162.1, U67.9
- removed net SCL17: J205.4, J206.4, J207.4, J214.3, R172.1, U71.9
- removed net SCL8: J106.3, J97.4, J98.4, J99.4, R82.1, U35.9
- removed net SCL9: J109.4, J110.4, J111.4, J118.3, R92.1, U39.9
- removed net SCL_PU10: JP118.1, R92.2
- removed net SCL_PU11: JP130.1, R102.2
- removed net SCL_PU12: JP142.1, R112.2
- removed net SCL_PU13: JP154.1, R122.2
- removed net SCL_PU14: JP166.1, R132.2
- removed net SCL_PU15: JP178.1, R142.2
- removed net SCL_PU16: JP190.1, R152.2
- removed net SCL_PU17: JP202.1, R162.2
- removed net SCL_PU18: JP214.1, R172.2
- removed net SCL_PU9: JP106.1, R82.2
- removed net SDA10: J121.3, J122.3, J123.3, J130.4, R103.1, U43.7
- removed net SDA11: J133.3, J134.3, J135.3, J142.4, R113.1, U47.7
- removed net SDA12: J145.3, J146.3, J147.3, J154.4, R123.1, U51.7
- removed net SDA13: J157.3, J158.3, J159.3, J166.4, R133.1, U55.7
- removed net SDA14: J169.3, J170.3, J171.3, J178.4, R143.1, U59.7
- removed net SDA15: J181.3, J182.3, J183.3, J190.4, R153.1, U63.7
- removed net SDA16: J193.3, J194.3, J195.3, J202.4, R163.1, U67.7
- removed net SDA17: J205.3, J206.3, J207.3, J214.4, R173.1, U71.7
- removed net SDA8: J106.4, J97.3, J98.3, J99.3, R83.1, U35.7
- removed net SDA9: J109.3, J110.3, J111.3, J118.4, R93.1, U39.7
- removed net SDA_PU10: JP118.3, R93.2
- removed net SDA_PU11: JP130.3, R103.2
- removed net SDA_PU12: JP142.3, R113.2
- removed net SDA_PU13: JP154.3, R123.2
- removed net SDA_PU14: JP166.3, R133.2
- removed net SDA_PU15: JP178.3, R143.2
- removed net SDA_PU16: JP190.3, R153.2
- removed net SDA_PU17: JP202.3, R163.2
- removed net SDA_PU18: JP214.3, R173.2
- removed net SDA_PU9: JP106.3, R83.2
- removed net SD_CLK10: J129.SCLK, R108.2, U41.9
- removed net SD_CLK11: J141.SCLK, R118.2, U45.9
- removed net SD_CLK12: J153.SCLK, R128.2, U49.9
- removed net SD_CLK13: J165.SCLK, R138.2, U53.9
- removed net SD_CLK14: J177.SCLK, R148.2, U57.9
- removed net SD_CLK15: J189.SCLK, R158.2, U61.9
- removed net SD_CLK16: J201.SCLK, R168.2, U65.9
- removed net SD_CLK17: J213.SCLK, R178.2, U69.9
- removed net SD_CLK8: J105.SCLK, R88.2, U33.9
- removed net SD_CLK9: J117.SCLK, R98.2, U37.9
- removed net SD_CMD10: J129.DI, U41.10
- removed net SD_CMD11: J141.DI, U45.10
- removed net SD_CMD12: J153.DI, U49.10
- removed net SD_CMD13: J165.DI, U53.10
- removed net SD_CMD14: J177.DI, U57.10
- removed net SD_CMD15: J189.DI, U61.10
- removed net SD_CMD16: J201.DI, U65.10
- removed net SD_CMD17: J213.DI, U69.10
- removed net SD_CMD8: J105.DI, U33.10
- removed net SD_CMD9: J117.DI, U37.10
- removed net SD_DAT10: J129.DO, U41.8
- removed net SD_DAT11: J141.DO, U45.8
- removed net SD_DAT12: J153.DO, U49.8
- removed net SD_DAT13: J165.DO, U53.8
- removed net SD_DAT14: J177.DO, U57.8
- removed net SD_DAT15: J189.DO, U61.8
- removed net SD_DAT16: J201.DO, U65.8
- removed net SD_DAT17: J213.DO, U69.8
- removed net SD_DAT8: J105.DO, U33.8
- removed net SD_DAT9: J117.DO, U37.8
- removed net TRIGGER33: J104.1, U35.10
- removed net TRIGGER34: J104.4, J106.1, U35.8
- removed net TRIGGER35: J104.2, U35.5
- removed net TRIGGER36: J104.3, U35.2
- removed net TRIGGER37: J116.1, U39.10
- removed net TRIGGER38: J116.4, J118.1, U39.8
- removed net TRIGGER39: J116.2, U39.5
- removed net TRIGGER40: J116.3, U39.2
- removed net TRIGGER41: J128.1, U43.10
- removed net TRIGGER42: J128.4, J130.1, U43.8
- removed net TRIGGER43: J128.2, U43.5
- removed net TRIGGER44: J128.3, U43.2
- removed net TRIGGER45: J140.1, U47.10
- removed net TRIGGER46: J140.4, J142.1, U47.8
- removed net TRIGGER47: J140.2, U47.5
- removed net TRIGGER48: J140.3, U47.2
- removed net TRIGGER49: J152.1, U51.10
- removed net TRIGGER50: J152.4, J154.1, U51.8
- removed net TRIGGER51: J152.2, U51.5
- removed net TRIGGER52: J152.3, U51.2
- removed net TRIGGER53: J164.1, U55.10
- removed net TRIGGER54: J164.4, J166.1, U55.8
- removed net TRIGGER55: J164.2, U55.5
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Routing:
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- removed copper zone on layer 1, net GND10
- removed copper zone on layer 16, net GND10
- removed copper zone on layer 1, net GND11
- removed copper zone on layer 16, net GND11
- removed copper zone on layer 1, net GND12
- removed copper zone on layer 16, net GND12
- removed copper zone on layer 1, net GND13
- removed copper zone on layer 16, net GND13
- removed copper zone on layer 1, net GND14
- removed copper zone on layer 16, net GND14
- removed copper zone on layer 1, net GND15
- removed copper zone on layer 16, net GND15
- removed copper zone on layer 1, net GND16
- removed copper zone on layer 16, net GND16
- removed copper zone on layer 1, net GND17
- removed copper zone on layer 16, net GND17
- removed copper zone on layer 1, net GND8
- removed copper zone on layer 16, net GND8
- removed copper zone on layer 1, net GND9
- removed copper zone on layer 16, net GND9
Other:
- board size 203.5 x 167.1 mm -> 143.5 x 115.8 mm
- board text added: "X02"
- board text removed: "X01"
