File: Hardware/Production/Qwiic MP3 Trigger-Panel.brd (EAGLE design)
At the start: 115.6 x 115.8 mm, 636 parts, among them J1 MICRO-SD, J13 PTH, J14 QWIIC_RIGHT_ANGLE, J2 QWIIC_RIGHT_ANGLE, J20 MICRO-SD, J21 ISP, J22 Poke-Home, J23 3.5mm Audio, J25 QWIIC_RIGHT_ANGLE, J26 PTH, J27 QWIIC_RIGHT_ANGLE, J3 PTH, J32 MICRO-SD, J33 ISP, J34 Poke-Home, J35 3.5mm Audio, J37 QWIIC_RIGHT_ANGLE, J38 PTH, J39 QWIIC_RIGHT_ANGLE, J4 QWIIC_RIGHT_ANGLE, J44 MICRO-SD, J45 ISP, J46 Poke-Home, J47 3.5mm Audio, J49 QWIIC_RIGHT_ANGLE, J50 PTH, J51 QWIIC_RIGHT_ANGLE, J56 MICRO-SD, J57 ISP, J58 Poke-Home, J59 3.5mm Audio, J6 QWIIC_RIGHT_ANGLE, J61 QWIIC_RIGHT_ANGLE, J62 PTH, J63 QWIIC_RIGHT_ANGLE, J68 MICRO-SD, J69 ISP, J7 ISP, J70 Poke-Home, J71 3.5mm Audio, J8 3.5mm Audio, J9 Poke-Home, U1 TPA2005D1, U10 ATTINY84-ARDUINO, U11 AP2112-3.3V, U12 WT2003SH4, U13 TPA2005D1, U14 ATTINY84-ARDUINO, U15 AP2112-3.3V, U16 WT2003SH4, U17 TPA2005D1, U18 ATTINY84-ARDUINO, U19 AP2112-3.3V, U2 TPA2005D1, U20 WT2003SH4, U21 TPA2005D1, U22 ATTINY84-ARDUINO, U23 AP2112-3.3V, U24 WT2003SH4, U3 AP2112-3.3V, U4 ATTINY84-ARDUINO, U5 WT2003SH4, U6 ATTINY84-ARDUINO, U7 AP2112-3.3V, U8 WT2003SH4, U9 TPA2005D1

Commit message: Proto with MY1690
Parts:
- removed U$283: (no value), Labels:QWIIC-LOGO-MEDIUM
- removed U$284: (no value), buzzard_labels (2):TRIGGER4
- removed U$285: (no value), buzzard_labels (3):MP31
- removed U$286: (no value), buzzard_labels (3):QWIIC0
- removed U$287: (no value), buzzard_labels (3):TRIGGER2
- removed U$288: (no value), output:#PWR#0
- added LOGO19, LOGO23: SFE_LOGO_NAME_FLAME.1_INCH, SparkFun-Aesthetics:SFE_LOGO_NAME_FLAME_.1
- added LOGO20, LOGO24: QWIIC_LOGO_CONNECTOR, SparkFun-Aesthetics:QWIIC_5.5MM
- added LOGO21: OSHW-LOGOMINI, SparkFun-Aesthetics:OSHW-LOGO-MINI
- added LOGO22: SFE_LOGO_NAME.1_INCH, SparkFun-Aesthetics:SFE_LOGO_NAME_.1
- C1, C11, C22, C32, C42, C52: value 10uF -> 1.0uF
- C15, C26, C36, C46, C5, C56: device SparkFun-Capacitors:0402 -> SparkFun-Capacitors:0603
- J1: value MICRO-SD -> QWIIC_RIGHT_ANGLE; device SparkFun-Connectors:MICRO-SD-SOCKET -> SparkFun-Connectors:JST04_1MM_RA
- J13: value PTH -> QWIIC_RIGHT_ANGLE; device SparkX:1X04_NO_SILK -> SparkFun-Connectors:JST04_1MM_RA
- J14: value QWIIC_RIGHT_ANGLE -> MICRO-SD; device SparkFun-Connectors:JST04_1MM_RA -> SparkFun-Connectors:MICROSD-EXTERNALPIN
- J20, J32, J44, J56, J68: value MICRO-SD -> ISP; device SparkFun-Connectors:MICRO-SD-SOCKET -> SparkFun-Connectors:2X3_TEST_POINTS
- J21, J33, J45, J57, J69: value ISP -> Poke-Home; device SparkFun-Connectors:2X3_TEST_POINTS -> SparkFun-Connectors:1X02_POKEHOME
- J22, J34, J46, J58, J70: value Poke-Home -> 3.5mm Audio; device SparkFun-Connectors:1X02_POKEHOME -> SparkFun-Connectors:AUDIO_JACK_3.5MM_TRRS_SMD_RA
- J23, J35, J47, J59, J71: value 3.5mm Audio -> (none); device SparkFun-Connectors:AUDIO_JACK_3.5MM_TRRS_SMD_RA -> SparkFun-Connectors:USB-C-16P-2LAYER-PADS
- J24, J36, J48, J60, J72: value (none) -> MICRO-SD; device SparkFun-Connectors:USB-C-16P-2LAYER-PADS -> SparkFun-Connectors:MICROSD-EXTERNALPIN
- J6: value QWIIC_RIGHT_ANGLE -> PTH; device SparkFun-Connectors:JST04_1MM_RA -> SparkX:1X04_NO_SILK
- LOGO10: value OSHW-LOGOMINI -> SFE_LOGO_NAME.1_INCH; device SparkFun-Aesthetics:OSHW-LOGO-MINI -> SparkFun-Aesthetics:SFE_LOGO_NAME_.1
- LOGO11: value SFE_LOGO_NAME.1_INCH -> SFE_LOGO_NAME_FLAME.1_INCH; device SparkFun-Aesthetics:SFE_LOGO_NAME_.1 -> SparkFun-Aesthetics:SFE_LOGO_NAME_FLAME_.1
- LOGO12: value SFE_LOGO_NAME_FLAME.1_INCH -> QWIIC_LOGO_CONNECTOR; device SparkFun-Aesthetics:SFE_LOGO_NAME_FLAME_.1 -> SparkFun-Aesthetics:QWIIC_5.5MM
- LOGO16, LOGO4: value OSHW-LOGOMINI -> QWIIC_LOGO_CONNECTOR; device SparkFun-Aesthetics:OSHW-LOGO-MINI -> SparkFun-Aesthetics:QWIIC_5.5MM
- LOGO17, LOGO5: value SFE_LOGO_NAME.1_INCH -> OSHW-LOGOMINI; device SparkFun-Aesthetics:SFE_LOGO_NAME_.1 -> SparkFun-Aesthetics:OSHW-LOGO-MINI
- LOGO18, LOGO6: value SFE_LOGO_NAME_FLAME.1_INCH -> SFE_LOGO_NAME.1_INCH; device SparkFun-Aesthetics:SFE_LOGO_NAME_FLAME_.1 -> SparkFun-Aesthetics:SFE_LOGO_NAME_.1
- LOGO7: value OSHW-LOGOMINI -> SFE_LOGO_NAME_FLAME.1_INCH; device SparkFun-Aesthetics:OSHW-LOGO-MINI -> SparkFun-Aesthetics:SFE_LOGO_NAME_FLAME_.1
- LOGO8: value SFE_LOGO_NAME.1_INCH -> QWIIC_LOGO_CONNECTOR; device SparkFun-Aesthetics:SFE_LOGO_NAME_.1 -> SparkFun-Aesthetics:QWIIC_5.5MM
- LOGO9: value SFE_LOGO_NAME_FLAME.1_INCH -> OSHW-LOGOMINI; device SparkFun-Aesthetics:SFE_LOGO_NAME_FLAME_.1 -> SparkFun-Aesthetics:OSHW-LOGO-MINI
- U$10, U$38, U$69: device buzzard_labels (16):#6 -> output:#1#3
- U$100, U$148: device Labels-0_04:SDA8 -> output:#0
- U$101, U$194, U$242: device Labels-0_04:GND1 -> output:#0
- U$102, U$150: device Labels-0_04:3#3V2 -> output:#1
- U$103, U$196, U$244: device Labels-0_04:SDA8 -> output:#1
- U$104: device Labels-0_04:SCL9 -> output:QWIIC_MP30
- U$105: device Labels:I_SUPER2_C-()-03 -> output:TRIGGER1
- U$106: device Labels:INT#-[< -> output:#PWR#0
- U$107, U$154, U$155, U$202: device Labels:INT#-[< -> output:TRIGGER0
- U$108: device Labels:RST#-[> -> output:TRIGGER0
- U$109, U$156, U$157, U$204: device Labels:RST#-[> -> output:L1
- U$11: device Labels:INT#-[< -> output:#1
- U$110: device Labels:PWR-()-03 -> output:L1
- U$111, U$159: device Labels:ADR-()-03 -> output:R0
- U$112, U$64: device buzzard_labels (13):TRIGGER5 -> output:R0
- U$113, U$161: device buzzard_labels (14):21 -> output:#2
- U$114, U$66: device buzzard_labels (14):32 -> output:#2
- U$115, U$163: device buzzard_labels (14):43 -> output:#1#3
- U$116, U$68: device buzzard_labels (16):#5 -> output:#1#3
- U$117, U$165: device buzzard_labels (16):#6 -> output:#2#2
- U$118, U$70: device buzzard_labels (16):1_1 -> output:#2#2
- U$119, U$167: device buzzard_labels (16):GND0 -> output:#3#1
- U$12, U$28: device buzzard_labels (16):#5 -> output:#1
- U$120, U$72: device buzzard_labels (16):L12 -> output:#3#1
- U$121, U$169: device buzzard_labels (16):R11 -> output:#4#0
- U$122, U$74: device buzzard_labels (16):#6 -> output:#4#0
- U$123, U$171: device buzzard_labels (17):PHONES0 -> output:#GND#0
- U$124, U$76: device buzzard_labels (17):SPEAKER1 -> output:#GND#0
- U$125: device buzzard_labels (17):QWIIC_MP32 -> output:PHONES0
- U$126: device buzzard_labels (16):#6 -> output:#PWR#0
- U$127: device buzzard_labels (16):#5 -> output:#ADR#0
- U$128: device buzzard_labels (14):43 -> output:SPEAKER0
- U$129: device buzzard_labels (14):32 -> output:#I�C#0
- U$13: device buzzard_labels (16):#6 -> output:#1
- U$130, U$178: device buzzard_labels (16):#6 -> output:##INT##4
- U$131, U$83: device buzzard_labels (16):R11 -> output:##INT##4
- U$132, U$180: device buzzard_labels (16):L12 -> output:##RST##5
- U$133, U$85: device buzzard_labels (14):21 -> output:##RST##5
- U$134, U$182, U$44: device buzzard_labels (16):1_1 -> output:#3#3V#0
- U$135, U$87: device buzzard_labels (13):TRIGGER5 -> output:#3#3V#0
- U$136, U$184, U$46: device buzzard_labels (16):GND0 -> output:#GND#1
- U$137, U$89: device buzzard_labels (17):PHONES0 -> output:#GND#1
- U$138, U$186: device buzzard_labels (17):SPEAKER1 -> output:#SCL#3
- U$139, U$91: device Labels:QWIIC-LOGO-MEDIUM -> output:#SCL#3
- U$14: device buzzard_labels (17):SPEAKER1 -> output:#0
- U$140, U$188: device buzzard_labels (2):TRIGGER4 -> output:#SDA#2
- U$141, U$93: device buzzard_labels (3):MP31 -> output:#SDA#2
- U$142: device buzzard_labels (3):QWIIC0 -> buzzard_labels (3):MP31
- U$143: device buzzard_labels (3):TRIGGER2 -> buzzard_labels (3):QWIIC0
- U$144: device output:#PWR#0 -> buzzard_labels (3):TRIGGER2
- U$145: device Labels-0_04:3#3V2 -> output:PHONES0
- U$146: device Labels-0_04:GND1 -> output:SPEAKER0
- U$147, U$195, U$51: device Labels-0_04:SCL9 -> output:#0
- U$149, U$197: device Labels-0_04:GND1 -> output:#1
- U$15, U$267: device buzzard_labels (17):PHONES0 -> output:#PWR#0
- U$151: device Labels-0_04:SDA8 -> output:QWIIC_MP30
- U$152: device Labels-0_04:SCL9 -> output:TRIGGER1
- U$153: device Labels:I_SUPER2_C-()-03 -> output:#PWR#0
- U$158, U$206: device Labels:PWR-()-03 -> output:R0
- U$16: device Labels:RST#-[> -> output:QWIIC_MP30
- U$160, U$208: device buzzard_labels (13):TRIGGER5 -> output:#2
- U$162, U$210: device buzzard_labels (14):32 -> output:#1#3
- U$164, U$212: device buzzard_labels (16):#5 -> output:#2#2
- U$166, U$214: device buzzard_labels (16):1_1 -> output:#3#1
- U$168, U$216: device buzzard_labels (16):L12 -> output:#4#0
- U$17: device Labels:PWR-()-03 -> output:#ADR#0
- U$170, U$218: device buzzard_labels (16):#6 -> output:#GND#0
- U$172: device buzzard_labels (17):SPEAKER1 -> output:PHONES0
- U$173, U$24: device buzzard_labels (17):QWIIC_MP32 -> output:#PWR#0
- U$174: device buzzard_labels (16):#6 -> output:#ADR#0
- U$175: device buzzard_labels (16):#5 -> output:SPEAKER0
- U$176: device buzzard_labels (14):43 -> output:#I�C#0
- U$177, U$225, U$33: device buzzard_labels (14):32 -> output:##INT##4
- U$179, U$227: device buzzard_labels (16):R11 -> output:##RST##5
- U$18: device Labels:ADR-()-03 -> output:SPEAKER0
- U$181, U$229, U$42: device buzzard_labels (14):21 -> output:#3#3V#0
- U$183, U$231: device buzzard_labels (13):TRIGGER5 -> output:#GND#1
- U$185, U$233: device buzzard_labels (17):PHONES0 -> output:#SCL#3
- U$187, U$235: device Labels:QWIIC-LOGO-MEDIUM -> output:#SDA#2
- U$19: device buzzard_labels (16):1_1 -> output:#GND#0
- U$192: device output:#PWR#0 -> output:PHONES0
- U$193: device Labels-0_04:3#3V2 -> output:SPEAKER0
- U$198: device Labels-0_04:3#3V2 -> output:QWIIC_MP30
- U$199, U$52: device Labels-0_04:SDA8 -> output:TRIGGER1
- U$2: device output:#PWR#0 -> output:TRIGGER0
- U$20: device buzzard_labels (17):SPEAKER1 -> output:#I�C#0
- U$200: device Labels-0_04:SCL9 -> output:#PWR#0
- U$201, U$249: device Labels:I_SUPER2_C-()-03 -> output:TRIGGER0
- U$203, U$250, U$251: device Labels:INT#-[< -> output:L1
- U$205, U$252, U$253: device Labels:RST#-[> -> output:R0
- U$207, U$255: device Labels:ADR-()-03 -> output:#2
- U$209, U$257: device buzzard_labels (14):21 -> output:#1#3
- U$21, U$246: device Labels-0_04:3#3V2 -> output:TRIGGER1
- U$211, U$259: device buzzard_labels (14):43 -> output:#2#2
- U$213, U$261: device buzzard_labels (16):#6 -> output:#3#1
- U$215, U$263: device buzzard_labels (16):GND0 -> output:#4#0
- U$217, U$265: device buzzard_labels (16):R11 -> output:#GND#0
- U$219: device buzzard_labels (17):PHONES0 -> output:PHONES0
- U$22: device Labels-0_04:GND1 -> output:#PWR#0
- U$220: device buzzard_labels (17):SPEAKER1 -> output:#PWR#0
- U$221: device buzzard_labels (17):QWIIC_MP32 -> output:#ADR#0
- U$222: device buzzard_labels (16):#6 -> output:SPEAKER0
- U$223: device buzzard_labels (16):#5 -> output:#I�C#0
- U$224, U$272, U$34: device buzzard_labels (14):43 -> output:##INT##4
- U$226, U$274: device buzzard_labels (16):#6 -> output:##RST##5
- U$228, U$276: device buzzard_labels (16):L12 -> output:#3#3V#0
- U$230, U$278: device buzzard_labels (16):1_1 -> output:#GND#1
- U$232, U$280: device buzzard_labels (16):GND0 -> output:#SCL#3
- U$234, U$282: device buzzard_labels (17):SPEAKER1 -> output:#SDA#2
- U$236: device buzzard_labels (2):TRIGGER4 -> buzzard_labels (3):MP31
- U$237: device buzzard_labels (3):MP31 -> buzzard_labels (3):QWIIC0
- U$238: device buzzard_labels (3):QWIIC0 -> buzzard_labels (3):TRIGGER2
- U$239: device buzzard_labels (3):TRIGGER2 -> output:PHONES0
- U$240: device output:#PWR#0 -> output:SPEAKER0
- U$241: device Labels-0_04:3#3V2 -> output:#0
- U$243: device Labels-0_04:SCL9 -> output:#1
- U$245: device Labels-0_04:GND1 -> output:QWIIC_MP30
- U$247: device Labels-0_04:SDA8 -> output:#PWR#0
- U$248, U$26: device Labels-0_04:SCL9 -> output:TRIGGER0
- U$25: device buzzard_labels (16):#6 -> output:QWIIC_MP30
- U$254: device Labels:PWR-()-03 -> output:#2
- U$256: device buzzard_labels (13):TRIGGER5 -> output:#1#3
- U$258: device buzzard_labels (14):32 -> output:#2#2
- U$260: device buzzard_labels (16):#5 -> output:#3#1
- U$262: device buzzard_labels (16):1_1 -> output:#4#0
- U$264: device buzzard_labels (16):L12 -> output:#GND#0
- U$266, U$78: device buzzard_labels (16):#6 -> output:PHONES0
- U$268: device buzzard_labels (17):SPEAKER1 -> output:#ADR#0
- U$269: device buzzard_labels (17):QWIIC_MP32 -> output:SPEAKER0
- U$27: device Labels-0_04:SDA8 -> output:TRIGGER0
- U$270, U$82: device buzzard_labels (16):#6 -> output:#I�C#0
- U$271: device buzzard_labels (16):#5 -> output:##INT##4
- U$273, U$36: device buzzard_labels (14):32 -> output:##RST##5
- U$275: device buzzard_labels (16):R11 -> output:#3#3V#0
- U$277: device buzzard_labels (14):21 -> output:#GND#1
- U$279: device buzzard_labels (13):TRIGGER5 -> output:#SCL#3
- U$281: device buzzard_labels (17):PHONES0 -> output:#SDA#2
- U$29, U$45: device buzzard_labels (13):TRIGGER5 -> output:L1
- U$3: device Labels-0_04:GND1 -> buzzard_labels (3):MP31
- U$30: device Labels-0_04:3#3V2 -> output:L1
- U$31: device buzzard_labels (14):43 -> output:#GND#0
- U$32: device buzzard_labels (14):21 -> output:PHONES0
- U$35: device buzzard_labels (16):GND0 -> output:##RST##5
- U$37: device buzzard_labels (16):L12 -> output:R0
- U$39: device buzzard_labels (16):R11 -> output:R0
- U$4: device Labels-0_04:3#3V2 -> buzzard_labels (3):QWIIC0
- U$40: device buzzard_labels (17):PHONES0 -> output:SPEAKER0
- U$41: device buzzard_labels (16):L12 -> output:#2
- U$43: device buzzard_labels (16):R11 -> output:#2
- U$47: device Labels:QWIIC-LOGO-MEDIUM -> output:TRIGGER0
- U$48, U$98: device Labels-0_04:GND1 -> output:PHONES0
- U$49: device buzzard_labels (2):TRIGGER4 -> output:#2#2
- U$5: device Labels-0_04:SDA8 -> buzzard_labels (3):TRIGGER2
- U$53: device Labels-0_04:GND1 -> output:#2#2
- U$54: device Labels-0_04:3#3V2 -> output:#3#1
- U$55: device Labels-0_04:SDA8 -> output:#3#1
- U$56: device Labels-0_04:SCL9 -> output:#4#0
- U$57: device Labels:I_SUPER2_C-()-03 -> output:#4#0
- U$58: device Labels:INT#-[< -> output:#GND#1
- U$59: device Labels:INT#-[< -> output:#SCL#3
- U$6: device Labels-0_04:SCL9 -> output:PHONES0
- U$60: device Labels:RST#-[> -> output:#SCL#3
- U$61: device Labels:RST#-[> -> output:#SDA#2
- U$62: device Labels:PWR-()-03 -> output:#SDA#2
- U$63: device Labels:ADR-()-03 -> output:L1
- U$65: device buzzard_labels (14):21 -> output:R0
- U$67: device buzzard_labels (14):43 -> output:#2
- U$7: device Labels:RST#-[> -> output:SPEAKER0
- U$71: device buzzard_labels (16):GND0 -> output:#2#2
- U$73: device buzzard_labels (16):R11 -> output:#3#1
- U$75: device buzzard_labels (17):PHONES0 -> output:#4#0
- U$77: device buzzard_labels (17):QWIIC_MP32 -> output:#GND#0
- U$79: device buzzard_labels (16):#5 -> output:#PWR#0
- U$8: device Labels:I_SUPER2_C-()-03 -> output:#0
- U$80: device buzzard_labels (14):43 -> output:#ADR#0
- U$81: device buzzard_labels (14):32 -> output:SPEAKER0
- U$84: device buzzard_labels (16):L12 -> output:##INT##4
- U$86: device buzzard_labels (16):1_1 -> output:##RST##5
- U$88: device buzzard_labels (16):GND0 -> output:#3#3V#0
- U$9: device Labels:INT#-[< -> output:#0
- U$90: device buzzard_labels (17):SPEAKER1 -> output:#GND#1
- U$92: device buzzard_labels (2):TRIGGER4 -> output:#SCL#3
- U$94: device buzzard_labels (3):QWIIC0 -> output:#SDA#2
- U$95: device buzzard_labels (3):TRIGGER2 -> buzzard_labels (3):MP31
- U$96: device output:#PWR#0 -> buzzard_labels (3):QWIIC0
- U$97: device Labels-0_04:3#3V2 -> buzzard_labels (3):TRIGGER2
- U$99: device Labels-0_04:SCL9 -> output:SPEAKER0
- U12, U16, U20, U24, U8: value WT2003SH4 -> MY1690-16S; device SparkFun-IC-Special-Function:SO16 -> MY1690:SO16
- U2: value TPA2005D1 -> MY1690-16S; device SparkFun-IC-Amplifiers:QFN-8_PAD -> MY1690:SO16
- U5: value WT2003SH4 -> TPA2005D1; device SparkFun-IC-Special-Function:SO16 -> SparkFun-IC-Amplifiers:QFN-8_PAD
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Connections:
- removed net N$13 (its old number): J24.B5, R24.2
- removed net N$21 (its old number): J36.B5, R37.2
- removed net N$22 (its old number): J36.A5, R38.2
- removed net N$29 (its old number): J48.B5, R50.2
- removed net N$30 (its old number): J48.A5, R51.2
- removed net N$37 (its old number): J60.B5, R63.2
- removed net N$38 (its old number): J60.A5, R64.2
- removed net N$46 (its old number): J72.A5, R77.2
- new net N$15: J23.A5, R25.2
- new net N$18: C12.1, U8.7
- new net N$23: J35.B5, R37.2
- new net N$24: J35.A5, R38.2
- new net N$27: C23.1, U12.7
- new net N$32: J47.B5, R50.2
- new net N$33: J47.A5, R51.2
- new net N$36: C33.1, U16.7
- new net N$41: J59.B5, R63.2
- new net N$42: J59.A5, R64.2
- new net N$50: J71.B5, R76.2
- new net N$51: J71.A5, R77.2
- new net N$54: C53.1, U24.7
- new net N$7: C4.1, U2.7
- net !RST1: now also J20.5; no longer J21.5
- net !RST2: now also J32.5; no longer J33.5
- net !RST3: now also J44.5; no longer J45.5
- net !RST4: now also J56.5; no longer J57.5
- net !RST5: now also J68.5; no longer J69.5
- net 3.3V: now also U2.12; no longer U5.11
- net 3.3V1: now also J1.2, J20.2, U5.6, U8.12; no longer J14.2, J21.2, U2.6, U8.11
- net 3.3V2: now also J32.2, U12.12; no longer J33.2, U12.11
- net 3.3V3: now also J44.2, U16.12; no longer J45.2, U16.11
- net 3.3V4: now also J56.2, U20.12; no longer J57.2, U20.11
- net 3.3V5: now also J68.2, U24.12; no longer J69.2, U24.11
- net 5V: now also C1.1; no longer C4.1
- net 5V1: now also C11.1, J23.VBUS1, J23.VBUS2; no longer C12.1, J24.VBUS1, J24.VBUS2
- net 5V2: now also C22.1, J35.VBUS1, J35.VBUS2; no longer C23.1, J36.VBUS1, J36.VBUS2
- net 5V3: now also C32.1, J47.VBUS1, J47.VBUS2; no longer C33.1, J48.VBUS1, J48.VBUS2
- net 5V4: now also C42.1, J59.VBUS1, J59.VBUS2; no longer C43.1, J60.VBUS1, J60.VBUS2
- net 5V5: now also C52.1, J71.VBUS1, J71.VBUS2; no longer C53.1, J72.VBUS1, J72.VBUS2
- net AC-L1: now also J22.RING1; no longer J23.RING1
- net AC-L2: now also J34.RING1; no longer J35.RING1
- net AC-L3: now also J46.RING1; no longer J47.RING1
- net AC-L4: now also J58.RING1; no longer J59.RING1
- net AC-L5: now also J70.RING1; no longer J71.RING1
- net AC-R1: now also J22.TIP; no longer J23.TIP
- net AC-R2: now also J34.TIP; no longer J35.TIP
- net AC-R3: now also J46.TIP; no longer J47.TIP
- net AC-R4: now also J58.TIP; no longer J59.TIP
- net AC-R5: now also J70.TIP; no longer J71.TIP
- net ADKEY: now also U2.4; no longer U5.7
- net ADKEY1: now also U8.4; no longer U8.7
- net ADKEY2: now also U12.4; no longer U12.7
- net ADKEY3: now also U16.4; no longer U16.7
- net ADKEY4: now also U20.4; no longer U20.7
- net ADKEY5: now also U24.4; no longer U24.7
- net D+: now also U2.6; no longer U5.5
- net D+1: now also J23.A6, J23.B6, U8.6; no longer J24.A6, J24.B6, U8.5
- net D+2: now also J35.A6, J35.B6, U12.6; no longer J36.A6, J36.B6, U12.5
- net D+3: now also J47.A6, J47.B6, U16.6; no longer J48.A6, J48.B6, U16.5
- net D+4: now also J59.A6, J59.B6, U20.6; no longer J60.A6, J60.B6, U20.5
- net D+5: now also J71.A6, J71.B6, U24.6; no longer J72.A6, J72.B6, U24.5
- net D-: now also U2.5; no longer U5.4
- net D-1: now also J23.A7, J23.B7, U8.5; no longer J24.A7, J24.B7, U8.4
- net D-2: now also J35.A7, J35.B7, U12.5; no longer J36.A7, J36.B7, U12.4
- net D-3: now also J47.A7, J47.B7, U16.5; no longer J48.A7, J48.B7, U16.4
- net D-4: now also J59.A7, J59.B7, U20.5; no longer J60.A7, J60.B7, U20.4
- net D-5: now also J71.A7, J71.B7, U24.5; no longer J72.A7, J72.B7, U24.4
- net GND: now also J14.10, J14.11, J14.12, J14.13, J14.6, U2.13, U2.8; no longer J1.CD1, J1.GND, U5.12, U5.8
- net GND1: now also J1.1, J20.6, J22.EARTH, J22.RING2, J23.GND, J23.GND2, J23.SHLD1, J23.SHLD2, J23.SHLD3, J23.SHLD4, J24.10, J24.11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; no longer J14.1, J20.CD1, J20.GND, J21.6, J23.EARTH, J23.RING2, J24.GND, J24.GND2, J24.SHLD1, J24.SHLD2, J24.SHLD3, J24.SHLD4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
- net GND2: now also J32.6, J34.EARTH, J34.RING2, J35.GND, J35.GND2, J35.SHLD1, J35.SHLD2, J35.SHLD3, J35.SHLD4, J36.10, J36.11, J36.12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; no longer J32.CD1, J32.GND, J33.6, J35.EARTH, J35.RING2, J36.GND, J36.GND2, J36.SHLD1, J36.SHLD2, J36.SHLD3, J36.SHLD4, U12.12
- net GND3: now also J44.6, J46.EARTH, J46.RING2, J47.GND, J47.GND2, J47.SHLD1, J47.SHLD2, J47.SHLD3, J47.SHLD4, J48.10, J48.11, J48.12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; no longer J44.CD1, J44.GND, J45.6, J47.EARTH, J47.RING2, J48.GND, J48.GND2, J48.SHLD1, J48.SHLD2, J48.SHLD3, J48.SHLD4, U16.12
- net GND4: now also J56.6, J58.EARTH, J58.RING2, J59.GND, J59.GND2, J59.SHLD1, J59.SHLD2, J59.SHLD3, J59.SHLD4, J60.10, J60.11, J60.12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; no longer J56.CD1, J56.GND, J57.6, J59.EARTH, J59.RING2, J60.GND, J60.GND2, J60.SHLD1, J60.SHLD2, J60.SHLD3, J60.SHLD4, U20.12
- net GND5: now also J68.6, J70.EARTH, J70.RING2, J71.GND, J71.GND2, J71.SHLD1, J71.SHLD2, J71.SHLD3, J71.SHLD4, J72.10, J72.11, J72.12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; no longer J68.CD1, J68.GND, J69.6, J71.EARTH, J71.RING2, J72.GND, J72.GND2, J72.SHLD1, J72.SHLD2, J72.SHLD3, J72.SHLD4, U24.12
- net IN+AMP1: now also U5.3; no longer U2.3
- net IN-AMP1: now also U5.4; no longer U2.4
- net MP3-RXI: now also U2.15; no longer U5.6
- net MP3-RXI1: now also U8.15; no longer U8.6
- net MP3-RXI2: now also U12.15; no longer U12.6
- net MP3-RXI3: now also U16.15; no longer U16.6
- net MP3-RXI4: now also U20.15; no longer U20.6
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Routing:
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Other:
- board text added: "v30"
- board text removed: "v20"

Commit message: Add v20 panel
Parts:
- added C100, C67, C78, C89: 0.1uF, SparkFun-Capacitors:0603
- added C101, C106, C109, C62, C65, C68, C73, C76, C79, C84, C87, C90, C95, C98: 1.0uF, SparkFun-Capacitors:0603
- added C102, C110, C66, C69, C77, C80, C88, C91, C99: 2.2uF, SparkFun-Capacitors:0603
- added C103, C104, C70, C71, C81, C82, C92, C93: 10nF, SparkFun-Capacitors:0603
- added C105, C61, C72, C83, C94: 22nF, SparkFun-Capacitors:0603
- added C107, C108, C63, C64, C74, C75, C85, C86, C96, C97: 0.22uF, SparkFun-Capacitors:0603
- added D10, D7, D8, D9: RED, SparkFun-LED:LED-0603
- added J100, J113, J126, J74, J87: Poke-Home, SparkFun-Connectors:1X02_POKEHOME
- added J101, J114, J127, J75, J88: 3.5mm Audio, SparkFun-Connectors:AUDIO_JACK_3.5MM_TRRS_SMD_RA
- added J102, J115, J128, J76, J89: (no value), SparkFun-Connectors:USB-C-16P-2LAYER-PADS
- added J103, J116, J129, J77, J90: MICRO-SD, SparkFun-Connectors:MICROSD-EXTERNALPIN
- added J104, J108, J109, J117, J121, J122, J130, J78, J82, J83, J91, J95, J96: (no value), SparkFun-Connectors:1X01_NO_SILK
- added J105, J107, J118, J120, J79, J81, J92, J94: QWIIC_RIGHT_ANGLE, SparkFun-Connectors:JST04_1MM_RA
- added J106, J119, J80, J93: PTH, SparkX:1X04_NO_SILK
- added J110, J111, J123, J124, J84, J85, J97, J98: (no value), SparkFun-Connectors:1X04_NO_SILK
- added J112, J125, J73, J86, J99: ISP, SparkFun-Connectors:2X3_TEST_POINTS
- added JP100, JP109, JP110, JP113, JP114, JP123, JP124, JP127, JP128, JP137, JP138, JP85, JP86, JP95, JP96, JP99: STAND-OFF, SparkFun:STAND-OFF
- added JP101, JP102, JP103, JP104, JP115, JP116, JP117, JP118, JP129, JP130, JP131, JP132, JP87, JP88, JP89, JP90: FIDUCIALUFIDUCIAL, SparkFun:MICRO-FIDUCIAL
- added JP105, JP119, JP133, JP91: PTH, SparkFun-Connectors:1X03_NO_SILK
- added JP106, JP120, JP134, JP92: PTH, SparkFun-Connectors:1X02_NO_SILK
- added JP107, JP121, JP135, JP93: ADR, SparkFun-Jumpers:SMT-JUMPER_2_NO_SILK
- added JP108, JP122, JP136, JP94: JUMPER-SMT_3_2-NC_TRACE_SILK, SparkFun-Jumpers:SMT-JUMPER_3_2-NC_TRACE_SILK
- added JP111, JP125, JP139, JP97: INT, SparkFun-Jumpers:SMT-JUMPER_2_NC_TRACE_SILK
- added JP112, JP126, JP140, JP98: JUMPER-SMT_2_NC_TRACE_SILK, SparkFun-Jumpers:SMT-JUMPER_2_NC_TRACE_SILK
- added LOGO25, LOGO29, LOGO33, LOGO37: OSHW-LOGOMINI, SparkFun-Aesthetics:OSHW-LOGO-MINI
- added LOGO26, LOGO30, LOGO34, LOGO38: SFE_LOGO_NAME.1_INCH, SparkFun-Aesthetics:SFE_LOGO_NAME_.1
- added LOGO27, LOGO31, LOGO35, LOGO39: SFE_LOGO_NAME_FLAME.1_INCH, SparkFun-Aesthetics:SFE_LOGO_NAME_FLAME_.1
- added LOGO28, LOGO32, LOGO36, LOGO40: QWIIC_LOGO_CONNECTOR, SparkFun-Aesthetics:QWIIC_5.5MM
- added R100, R101, R108, R112, R113, R120, R84, R88, R89, R96: 10k, SparkFun-Resistors:0603
- added R102, R114, R90: 47k, SparkFun-Resistors:0603
- added R103, R110, R111, R115, R79, R86, R87, R91, R98, R99: 2.2k, SparkFun-Resistors:0603
- added R104, R105, R116, R117, R80, R81, R92, R93: 100k, SparkFun-Resistors:0603
- added R106, R107, R118, R119, R82, R83, R94, R95: 5.1k, SparkFun-Resistors:0603
- added R109, R85, R97: 1k, SparkFun-Resistors:0603
- added U$283, U$330, U$331, U$378, U$379, U$426, U$427, U$474, U$475: (no value), output:#GND#1
- added U$284, U$285, U$332, U$333, U$380, U$381, U$428, U$429, U$476, U$477: (no value), output:#SCL#3
- added U$286, U$287, U$334, U$335, U$382, U$383, U$430, U$431, U$478, U$479: (no value), output:#SDA#2
- added U$288, U$336, U$384, U$432, U$480: (no value), output:#5V#0
- added U$289, U$337, U$385, U$433: (no value), buzzard_labels (3):MP31
- added U$290, U$338, U$386, U$434: (no value), buzzard_labels (3):QWIIC0
- added U$291, U$339, U$387, U$435: (no value), buzzard_labels (3):TRIGGER2
- added U$292, U$319, U$340, U$367, U$388, U$415, U$436, U$463: (no value), output:PHONES0
- added U$293, U$322, U$341, U$370, U$389, U$418, U$437, U$466: (no value), output:SPEAKER0
- added U$294, U$295, U$342, U$343, U$390, U$391, U$438, U$439: (no value), output:#0
- added U$296, U$297, U$344, U$345, U$392, U$393, U$440, U$441: (no value), output:#1
- added U$298, U$346, U$394, U$442: (no value), output:QWIIC_MP30
- added U$299, U$347, U$395, U$443: (no value), output:TRIGGER1
- added U$300, U$320, U$348, U$368, U$396, U$416, U$444, U$464: (no value), output:#PWR#0
- added U$301, U$302, U$349, U$350, U$397, U$398, U$445, U$446: (no value), output:TRIGGER0
- added U$303, U$304, U$351, U$352, U$399, U$400, U$447, U$448: (no value), output:L1
- added U$305, U$306, U$353, U$354, U$401, U$402, U$449, U$450: (no value), output:R0
- added U$307, U$308, U$355, U$356, U$403, U$404, U$451, U$452: (no value), output:#2
- added U$309, U$310, U$357, U$358, U$405, U$406, U$453, U$454: (no value), output:#1#3
- added U$311, U$312, U$359, U$360, U$407, U$408, U$455, U$456: (no value), output:#2#2
- added U$313, U$314, U$361, U$362, U$409, U$410, U$457, U$458: (no value), output:#3#1
- added U$315, U$316, U$363, U$364, U$411, U$412, U$459, U$460: (no value), output:#4#0
- added U$317, U$318, U$365, U$366, U$413, U$414, U$461, U$462: (no value), output:#GND#0
- added U$321, U$369, U$417, U$465: (no value), output:#ADR#0
- added U$323, U$371, U$419, U$467: (no value), output:#I�C#0
- added U$324, U$325, U$372, U$373, U$420, U$421, U$468, U$469: (no value), output:##INT##4
- added U$326, U$327, U$374, U$375, U$422, U$423, U$470, U$471: (no value), output:##RST##5
- added U$328, U$329, U$376, U$377, U$424, U$425, U$472, U$473: (no value), output:#3#3V#0
- added U25, U29, U33, U37: TPA2005D1, SparkFun-IC-Amplifiers:QFN-8_PAD
- added U26, U30, U34, U38: ATTINY84-ARDUINO, SparkFun-IC-Microcontroller:SO14
- added U27, U31, U35, U39: AP2112-3.3V, SparkFun-PowerIC:SOT23-5
- added U28, U32, U36, U40: MY1690X-16S, MY1690X-16S:SO16
- C10: value 0.1uF -> 2.2uF
- C11, C23: value 1.0uF -> 0.1uF
- C13, C25, C44, C55: value 10nF -> 2.2uF
- C15, C26: value 22nF -> 10nF
- C17, C50: value 1.0uF -> 22nF
- C18, C29: value 0.22uF -> 1.0uF
- C20, C30, C42, C52, C53: value 1.0uF -> 0.22uF
- C21, C51: value 0.1uF -> 1.0uF
- C22, C33, C4, C47: value 1.0uF -> 2.2uF
- C24, C35, C54: value 10nF -> 1.0uF
- C27, C37, C60: value 1.0uF -> 10nF
- C28, C39: value 0.22uF -> 22nF
- C31, C41: value 0.1uF -> 0.22uF
- C34, C45: value 10nF -> 0.1uF
- C36: value 22nF -> 2.2uF
- C38, C48, C49, C59: value 0.22uF -> 10nF
- C46: value 22nF -> 1.0uF
- C56: value 22nF -> 0.1uF
- C58: value 0.22uF -> 2.2uF
- J1, J39: value QWIIC_RIGHT_ANGLE -> (none); device SparkFun-Connectors:JST04_1MM_RA -> SparkFun-Connectors:1X01_NO_SILK
- J13: value QWIIC_RIGHT_ANGLE -> PTH; device SparkFun-Connectors:JST04_1MM_RA -> SparkX:1X04_NO_SILK
- J16, J29, J40, J53: value (none) -> QWIIC_RIGHT_ANGLE; device SparkFun-Connectors:1X01_NO_SILK -> SparkFun-Connectors:JST04_1MM_RA
- J18, J30, J31, J43: device SparkFun-Connectors:1X04_NO_SILK -> SparkFun-Connectors:1X01_NO_SILK
- J20, J32: value ISP -> (none); device SparkFun-Connectors:2X3_TEST_POINTS -> SparkFun-Connectors:1X04_NO_SILK
- J21: value Poke-Home -> ISP; device SparkFun-Connectors:1X02_POKEHOME -> SparkFun-Connectors:2X3_TEST_POINTS
- J22: value 3.5mm Audio -> Poke-Home; device SparkFun-Connectors:AUDIO_JACK_3.5MM_TRRS_SMD_RA -> SparkFun-Connectors:1X02_POKEHOME
- J23: value (none) -> 3.5mm Audio; device SparkFun-Connectors:USB-C-16P-2LAYER-PADS -> SparkFun-Connectors:AUDIO_JACK_3.5MM_TRRS_SMD_RA
- J24: value MICRO-SD -> (none); device SparkFun-Connectors:MICROSD-EXTERNALPIN -> SparkFun-Connectors:USB-C-16P-2LAYER-PADS
- J25, J51: value QWIIC_RIGHT_ANGLE -> MICRO-SD; device SparkFun-Connectors:JST04_1MM_RA -> SparkFun-Connectors:MICROSD-EXTERNALPIN
- J26: value PTH -> (none); device SparkX:1X04_NO_SILK -> SparkFun-Connectors:1X01_NO_SILK
- J28, J41: value (none) -> PTH; device SparkFun-Connectors:1X01_NO_SILK -> SparkX:1X04_NO_SILK
- J33, J45: value Poke-Home -> (none); device SparkFun-Connectors:1X02_POKEHOME -> SparkFun-Connectors:1X04_NO_SILK
- J34: value 3.5mm Audio -> ISP; device SparkFun-Connectors:AUDIO_JACK_3.5MM_TRRS_SMD_RA -> SparkFun-Connectors:2X3_TEST_POINTS
- J35: value (none) -> Poke-Home; device SparkFun-Connectors:USB-C-16P-2LAYER-PADS -> SparkFun-Connectors:1X02_POKEHOME
- J36: value MICRO-SD -> 3.5mm Audio; device SparkFun-Connectors:MICROSD-EXTERNALPIN -> SparkFun-Connectors:AUDIO_JACK_3.5MM_TRRS_SMD_RA
- J37, J63: value QWIIC_RIGHT_ANGLE -> (none); device SparkFun-Connectors:JST04_1MM_RA -> SparkFun-Connectors:USB-C-16P-2LAYER-PADS
- J38: value PTH -> MICRO-SD; device SparkX:1X04_NO_SILK -> SparkFun-Connectors:MICROSD-EXTERNALPIN
- J42, J55, J66: value (none) -> QWIIC_RIGHT_ANGLE; device SparkFun-Connectors:1X04_NO_SILK -> SparkFun-Connectors:JST04_1MM_RA
- J44, J56: value ISP -> (none); device SparkFun-Connectors:2X3_TEST_POINTS -> SparkFun-Connectors:1X01_NO_SILK
- J46, J58: value 3.5mm Audio -> (none); device SparkFun-Connectors:AUDIO_JACK_3.5MM_TRRS_SMD_RA -> SparkFun-Connectors:1X04_NO_SILK
- J47: value (none) -> ISP; device SparkFun-Connectors:USB-C-16P-2LAYER-PADS -> SparkFun-Connectors:2X3_TEST_POINTS
- J48: value MICRO-SD -> Poke-Home; device SparkFun-Connectors:MICROSD-EXTERNALPIN -> SparkFun-Connectors:1X02_POKEHOME
- J49: value QWIIC_RIGHT_ANGLE -> 3.5mm Audio; device SparkFun-Connectors:JST04_1MM_RA -> SparkFun-Connectors:AUDIO_JACK_3.5MM_TRRS_SMD_RA
- J50: value PTH -> (none); device SparkX:1X04_NO_SILK -> SparkFun-Connectors:USB-C-16P-2LAYER-PADS
- J54, J67: value (none) -> PTH; device SparkFun-Connectors:1X04_NO_SILK -> SparkX:1X04_NO_SILK
- J57, J69: value Poke-Home -> (none); device SparkFun-Connectors:1X02_POKEHOME -> SparkFun-Connectors:1X01_NO_SILK
- J59, J71: device SparkFun-Connectors:USB-C-16P-2LAYER-PADS -> SparkFun-Connectors:1X04_NO_SILK
- J6: value PTH -> QWIIC_RIGHT_ANGLE; device SparkX:1X04_NO_SILK -> SparkFun-Connectors:JST04_1MM_RA
- J60: value MICRO-SD -> ISP; device SparkFun-Connectors:MICROSD-EXTERNALPIN -> SparkFun-Connectors:2X3_TEST_POINTS
- J61: value QWIIC_RIGHT_ANGLE -> Poke-Home; device SparkFun-Connectors:JST04_1MM_RA -> SparkFun-Connectors:1X02_POKEHOME
- J62: value PTH -> 3.5mm Audio; device SparkX:1X04_NO_SILK -> SparkFun-Connectors:AUDIO_JACK_3.5MM_TRRS_SMD_RA
- J64: value (none) -> MICRO-SD; device SparkFun-Connectors:1X01_NO_SILK -> SparkFun-Connectors:MICROSD-EXTERNALPIN
- J68: value ISP -> QWIIC_RIGHT_ANGLE; device SparkFun-Connectors:2X3_TEST_POINTS -> SparkFun-Connectors:JST04_1MM_RA
- J70: value 3.5mm Audio -> (none); device SparkFun-Connectors:AUDIO_JACK_3.5MM_TRRS_SMD_RA -> SparkFun-Connectors:1X01_NO_SILK
- J72: value MICRO-SD -> (none); device SparkFun-Connectors:MICROSD-EXTERNALPIN -> SparkFun-Connectors:1X04_NO_SILK
- R1: value 10k -> 1k
- R12, R27: value 1k -> 2.2k
- R16, R28, R29, R41, R60: value 2.2k -> 10k
- R18, R30, R78: value 10k -> 47k
- R19: value 47k -> 2.2k
- R20, R33, R44, R56, R57, R69: value 10k -> 100k
- R21, R68: value 2.2k -> 100k
- R22, R23, R35: value 100k -> 5.1k
- R24, R64, R76, R77: value 5.1k -> 10k
- R25, R37: value 5.1k -> 1k
- R26, R31, R39, R43: value 10k -> 2.2k
- R32, R45: value 47k -> 100k
- R34, R47: value 2.2k -> 5.1k
- R36, R48: value 100k -> 10k
- R38, R50, R51, R63: value 5.1k -> 2.2k
- R40, R53: value 1k -> 10k
- R42, R54: value 2.2k -> 47k
- R46, R59, R70: value 10k -> 5.1k
- R49, R61: value 100k -> 1k
- R58, R71: value 47k -> 5.1k
- R62, R74, R75: value 100k -> 2.2k
- R66: value 1k -> 47k
- R73: value 2.2k -> 1k
- U$100, U$148: device output:#0 -> output:PHONES0
- U$101, U$8: device output:#0 -> output:SPEAKER0
- U$102, U$103, U$11, U$150: device output:#1 -> output:#0
- U$104, U$16: device output:QWIIC_MP30 -> output:#1
- U$105, U$152: device output:TRIGGER1 -> output:#1
- U$106: device output:#PWR#0 -> output:QWIIC_MP30
- U$107, U$155: device output:TRIGGER0 -> output:TRIGGER1
- U$108, U$26: device output:TRIGGER0 -> output:#PWR#0
- U$109, U$110, U$157, U$30: device output:L1 -> output:TRIGGER0
- U$111, U$112, U$159, U$64: device output:R0 -> output:L1
- U$113, U$114, U$161, U$66: device output:#2 -> output:R0
- U$115, U$116, U$163, U$68: device output:#1#3 -> output:#2
- U$117, U$118, U$165, U$70: device output:#2#2 -> output:#1#3
- U$119, U$120, U$167, U$72: device output:#3#1 -> output:#2#2
- U$121, U$122, U$169, U$74: device output:#4#0 -> output:#3#1
- U$123, U$124, U$171, U$76: device output:#GND#0 -> output:#4#0
- U$125, U$78: device output:PHONES0 -> output:#GND#0
- U$126, U$173: device output:#PWR#0 -> output:#GND#0
- U$127: device output:#ADR#0 -> output:PHONES0
- U$128: device output:SPEAKER0 -> output:#PWR#0
- U$129: device output:#I�C#0 -> output:#ADR#0
- U$130, U$178: device output:##INT##4 -> output:SPEAKER0
- U$131, U$83: device output:##INT##4 -> output:#I�C#0
- U$132, U$133, U$180, U$85: device output:##RST##5 -> output:##INT##4
- U$134, U$135, U$182, U$87: device output:#3#3V#0 -> output:##RST##5
- U$136, U$137, U$184, U$89: device output:#GND#1 -> output:#3#3V#0
- U$138, U$139, U$186, U$91: device output:#SCL#3 -> output:#GND#1
- U$140, U$141, U$188, U$93: device output:#SDA#2 -> output:#SCL#3
- U$142, U$95: device buzzard_labels (3):MP31 -> output:#SDA#2
- U$143, U$190: device buzzard_labels (3):QWIIC0 -> output:#SDA#2
- U$144: device buzzard_labels (3):TRIGGER2 -> output:#5V#0
- U$145: device output:PHONES0 -> buzzard_labels (3):MP31
- U$146: device output:SPEAKER0 -> buzzard_labels (3):QWIIC0
- U$147, U$195: device output:#0 -> buzzard_labels (3):TRIGGER2
- U$149, U$197: device output:#1 -> output:SPEAKER0
- U$151, U$198: device output:QWIIC_MP30 -> output:#0
- U$153, U$200: device output:#PWR#0 -> output:#1
- U$154, U$202: device output:TRIGGER0 -> output:QWIIC_MP30
- U$156, U$204: device output:L1 -> output:#PWR#0
- U$158, U$205, U$206, U$253: device output:R0 -> output:TRIGGER0
- U$160, U$207, U$208, U$255: device output:#2 -> output:L1
- U$162, U$209, U$210, U$257: device output:#1#3 -> output:R0
- U$164, U$211, U$212, U$259: device output:#2#2 -> output:#2
- U$166, U$213, U$214, U$261: device output:#3#1 -> output:#1#3
- U$168, U$215, U$216, U$263: device output:#4#0 -> output:#2#2
- U$170, U$217, U$218, U$265: device output:#GND#0 -> output:#3#1
- U$172, U$219: device output:PHONES0 -> output:#4#0
- U$174, U$221: device output:#ADR#0 -> output:#GND#0
- U$175, U$7: device output:SPEAKER0 -> output:PHONES0
- U$176: device output:#I�C#0 -> output:#PWR#0
- U$177, U$225: device output:##INT##4 -> output:#ADR#0
- U$179, U$227: device output:##RST##5 -> output:#I�C#0
- U$181, U$228, U$229, U$276: device output:#3#3V#0 -> output:##INT##4
- U$183, U$230, U$231, U$278: device output:#GND#1 -> output:##RST##5
- U$185, U$232, U$233, U$280: device output:#SCL#3 -> output:#3#3V#0
- U$187, U$234, U$235, U$282: device output:#SDA#2 -> output:#GND#1
- U$189, U$236: device buzzard_labels (3):MP31 -> output:#SCL#3
- U$191, U$238: device buzzard_labels (3):TRIGGER2 -> output:#SDA#2
- U$192: device output:PHONES0 -> output:#5V#0
- U$193: device output:SPEAKER0 -> buzzard_labels (3):MP31
- U$194, U$242: device output:#0 -> buzzard_labels (3):QWIIC0
- U$196, U$244: device output:#1 -> output:PHONES0
- U$199, U$246: device output:TRIGGER1 -> output:#0
- U$201, U$248, U$249: device output:TRIGGER0 -> output:#1
- U$203, U$251: device output:L1 -> output:TRIGGER1
- U$21: device output:TRIGGER1 -> output:QWIIC_MP30
- U$22: device output:#PWR#0 -> output:TRIGGER1
- U$220, U$267: device output:#PWR#0 -> output:#4#0
- U$222, U$269: device output:SPEAKER0 -> output:#GND#0
- U$223: device output:#I�C#0 -> output:PHONES0
- U$224, U$272: device output:##INT##4 -> output:#PWR#0
- U$226, U$274: device output:##RST##5 -> output:SPEAKER0
- U$237: device buzzard_labels (3):QWIIC0 -> output:#SCL#3
- U$239: device output:PHONES0 -> output:#SDA#2
- U$240: device output:SPEAKER0 -> output:#5V#0
- U$241: device output:#0 -> buzzard_labels (3):MP31
- U$243: device output:#1 -> buzzard_labels (3):TRIGGER2
- U$245: device output:QWIIC_MP30 -> output:SPEAKER0
- U$247: device output:#PWR#0 -> output:#0
- U$250: device output:L1 -> output:QWIIC_MP30
- U$252: device output:R0 -> output:#PWR#0
- U$254: device output:#2 -> output:TRIGGER0
- U$256: device output:#1#3 -> output:L1
- U$258: device output:#2#2 -> output:R0
- U$260: device output:#3#1 -> output:#2
- U$262: device output:#4#0 -> output:#1#3
- U$264: device output:#GND#0 -> output:#2#2
- U$266: device output:PHONES0 -> output:#3#1
- U$268: device output:#ADR#0 -> output:#4#0
- U$270: device output:#I�C#0 -> output:#GND#0
- U$271: device output:##INT##4 -> output:PHONES0
- U$273: device output:##RST##5 -> output:#ADR#0
- U$275: device output:#3#3V#0 -> output:#I�C#0
- U$277: device output:#GND#1 -> output:##INT##4
- U$279: device output:#SCL#3 -> output:##RST##5
- U$281: device output:#SDA#2 -> output:#3#3V#0
- U$3: device buzzard_labels (3):MP31 -> output:#5V#0
- U$4: device buzzard_labels (3):QWIIC0 -> buzzard_labels (3):MP31
- U$5: device buzzard_labels (3):TRIGGER2 -> buzzard_labels (3):QWIIC0
- U$6: device output:PHONES0 -> buzzard_labels (3):TRIGGER2
- U$79: device output:#PWR#0 -> output:PHONES0
- U$80: device output:#ADR#0 -> output:#PWR#0
- U$81: device output:SPEAKER0 -> output:#ADR#0
- U$82: device output:#I�C#0 -> output:SPEAKER0
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Connections:
- removed net ADKEY: R1.1, U2.4
- removed net ADKEY1: R20.1, U8.4
- removed net ADKEY2: R33.1, U12.4
- removed net ADKEY3: R46.1, U16.4
- removed net ADKEY4: R59.1, U20.4
- removed net ADKEY5: R72.1, U24.4
- removed net N$23 (its old number): J35.B5, R37.2
- new net !INT6: J82.1, R84.1, U26.6
- new net !INT7: J95.1, R96.1, U30.6
- new net !INT8: J108.1, R108.1, U34.6
- new net !INT9: J121.1, R120.1, U38.6
- new net !RST6: J83.1, J86.5, R76.1, U26.4
- new net !RST7: J96.1, J99.5, R88.1, U30.4
- new net !RST8: J109.1, J112.5, R100.1, U34.4
- new net !RST9: J122.1, J125.5, R112.1, U38.4
- new net 3.3V6: C67.1, C73.1, J79.2, J80.2, J81.2, J86.2, JP94.2, JP97.2, JP98.2, R76.2, R77.2, U25.6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
- new net 3.3V7: C78.1, C84.1, J92.2, J93.2, J94.2, J99.2, JP108.2, JP111.2, JP112.2, R88.2, R89.2, U29.6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
- new net 3.3V8: C89.1, C95.1, J105.2, J106.2, J107.2, J112.2, JP122.2, JP125.2, JP126.2, R100.2, R101.2, U33.6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
- new net 3.3V9: C100.1, C106.1, J118.2, J119.2, J120.2, J125.2, JP136.2, JP139.2, JP140.2, R112.2, R113.2, U37.6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
- new net 5V6: C68.1, J89.VBUS1, J89.VBUS2, J91.1, U27.1, U27.3
- new net 5V7: C79.1, J102.VBUS1, J102.VBUS2, J104.1, U31.1, U31.3
- new net 5V8: C90.1, J115.VBUS1, J115.VBUS2, J117.1, U35.1, U35.3
- new net 5V9: C101.1, J128.VBUS1, J128.VBUS2, J130.1, U39.1, U39.3
- new net AC-L6: C74.2, J88.RING1, JP91.3
- new net AC-L7: C85.2, J101.RING1, JP105.3
- new net AC-L8: C96.2, J114.RING1, JP119.3
- new net AC-L9: C107.2, J127.RING1, JP133.3
- new net AC-R6: C75.2, J88.TIP, JP91.2
- new net AC-R7: C86.2, J101.TIP, JP105.2
- new net AC-R8: C97.2, J114.TIP, JP119.2
- new net AC-R9: C108.2, J127.TIP, JP133.2
- new net ADR6: JP93.2, U26.3
- new net ADR7: JP107.2, U30.3
- new net ADR8: JP121.2, U34.3
- new net ADR9: JP135.2, U38.3
- new net D+6: J89.A6, J89.B6, U28.11
- new net D+7: J102.A6, J102.B6, U32.11
- new net D+8: J115.A6, J115.B6, U36.11
- new net D+9: J128.A6, J128.B6, U40.11
- new net D-6: J89.A7, J89.B7, U28.10
- new net D-7: J102.A7, J102.B7, U32.10
- new net D-8: J115.A7, J115.B7, U36.10
- new net D-9: J128.A7, J128.B7, U40.10
- new net GND6: C67.2, C68.2, C69.2, C72.1, C73.2, C76.2, C77.2, D7.C, J79.1, J80.1, J81.1, J84.1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
- new net GND7: C78.2, C79.2, C80.2, C83.1, C84.2, C87.2, C88.2, D8.C, J101.EARTH, J101.RING2, J102.GND, J102.GND2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
Routing:
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- added copper zone on layer 1, net GND6
- added copper zone on layer 16, net GND6
- added copper zone on layer 1, net GND7
- added copper zone on layer 16, net GND7
- added copper zone on layer 1, net GND8
- added copper zone on layer 16, net GND8
- added copper zone on layer 1, net GND9
- added copper zone on layer 16, net GND9
Other:
- board size 115.6 x 115.8 mm -> 176.5 x 115.8 mm
- board text added: "v20"
- board text removed: "v30"
