File: Hardware/MP3 Breakout.sch (EAGLE design)
At the start: 53 parts, among them J1 MICRO-SD, J3 PTH, J7 ISP, J8 3.5mm Audio, J9 Poke-Home, U1 TPA2005D1, U2 WT2003S, U3 AP2112-3.3V, U4 ATTINY84-ARDUINO

Commit message: OddCommit
Parts:
- removed C16: 1.0uF, SparkFun-Capacitors:1.0UF-16V-10%(0603)
- removed C2: 0.1uF, SparkFun-Capacitors:0.1UF-0603-25V-(+80/-20%)
- removed J10, J5: (no value), SparkFun-Connectors:CONN_01PTH_NO_SILK_YES_STOP
- removed J11, J12: (no value), SparkFun-Connectors:CONN_041X04_NO_SILK
- removed J7: ISP, SparkFun-Connectors:AVR_SPI_PROG_3X2TESTPOINTS
- removed J9: Poke-Home, SparkFun-Connectors:CONN_02SMALL_POKEHOME
- removed JP7: ADR, SparkFun-Jumpers:JUMPER-SMT_2_NO_NO-SILK
- removed JP9: JUMPER-SMT_3_2-NC_TRACE_SILK, SparkFun-Jumpers:JUMPER-SMT_3_2-NC_TRACE_SILK
- removed R3: 1k, SparkFun-Resistors:1KOHM-0603-1/10W-1%
- removed R6: 2.2k, SparkFun-Resistors:2.2KOHM-0603-1/10W-1%
- removed R8: 4.7k, SparkFun-Resistors:4.7KOHM-0603-1/10W-1%
- removed U$1: SPARKX-LOGO3, SparkX:SPARKX-LOGO3
- removed U3: AP2112-3.3V, SparkFun-PowerIC:V_REG_AP2112K-3.3V
- removed U4: ATTINY84-ARDUINO, SparkFun-IC-Microcontroller:ATTINY84-ARDUINO
- C9: device SparkFun-Capacitors:1.0UF-16V-10%(0603) -> SparkFun-Capacitors:1.0UF-0603-16V-10%
- J2: value (none) -> Header; device SparkFun-Connectors:QWIIC_CONNECTORJS-1MM -> SparkFun-Connectors:CONN_041X04_NO_SILK
- J3: value PTH -> (none); device SparkX:I2C_STANDARD_NO_SILK -> SparkFun-Connectors:CONN_01PTH_NO_SILK_YES_STOP
- J4: value (none) -> Poke-Home; device SparkFun-Connectors:QWIIC_CONNECTORJS-1MM -> SparkFun-Connectors:CONN_02SMALL_POKEHOME
- R2: value 2.2k -> 1k; device SparkFun-Resistors:2.2KOHM-0603-1/10W-1% -> SparkFun-Resistors:1KOHM-0603-1/10W-1%
Connections:
- removed net !INT: J5.1, U4.(A7)~7
- removed net !RST: J10.1, J7.5, R8.1, U4.(!RESET!)11
- removed net 3.3V: C16.1, C2.1, J2.2, J3.VCC, J4.2, J7.2, JP9.2, R10.2, R3.2, R8.2, U1.VDD, U2.VDDLDO, U3.OUT, U4.VCC
- removed net ADR: JP7.2, U4.(XTAL2)9
- removed net N$3: D1.A, R3.1
- removed net PLAYING: U2.BUSY, U4.(A2)2
- removed net SCL: J2.4, J3.SCL, J4.4, J7.3, R2.1, U4.(SCL/SCK/A4)4
- removed net SCL_PU1: JP9.1, R2.2
- removed net SDA: J2.3, J3.SDA, J4.3, J7.4, R6.1, U4.(RX/SDA/MOSI/A6)~6
- removed net SDA_PU1: JP9.3, R6.2
- removed net TRIGGER1: J12.4, J7.1, U4.(TX/MISO/A5)~5
- removed net TRIGGER2: J12.3, U4.(XTAL1)10
- removed net TRIGGER3: J12.2, U4.(INT0)~8
- removed net TRIGGER4: J12.1, U4.(A3)3
- new net N$1: D1.C, R2.2
- new net SHLD: J6.SHIELD
- net !SDN: now also J3.1, U2.BUSY; no longer U2.P10
- net 5V: now also D1.A, J2.3, U1.VDD, U2.VDDLDO; no longer U3.EN, U3.IN
- net GND: now also J2.4, R2.1; no longer C16.2, C2.2, D1.C, J11.1, J11.2, J11.3, J11.4, J2.1, J3.GND, J4.1, J6.SHIELD, J7.6, JP7.1, U3.GND, U4.GND
- net MP3-RXI: now also J2.2; no longer U4.(A0)0
- net MP3-TXO: now also J2.1; no longer U4.(A1)1
- net OUT+: now also J4.2; no longer J9.1
- net OUT-: now also J4.1; no longer J9.2
- net VCCIO: now also R10.2
Other:
- note added: "Note: This board has the supply labelled as 5V in order to prevent confusion when plugged into USB. It is possible to power the board from 3V3 but keep in mind that using both 3V3 and USB is not a good idea."
- note added: "O. Lyke"
- note added: "VDD upper limit 6V"
- note added: "VIN 3.0V to 5.5V, has onboard regulator that can supply 150 mA"
- note added: "X01"
- note removed: "3.3V 600mA Out"
- note removed: "3.3V VReg prevents USB 5V from being injected onto Qwiic 3.3V"
- note removed: "7-Bit Unshifted I2C Address Open Jumper (Default): 0x37 Closed Jumper: 0x36 Software configurable as well"
- note removed: "AVR"
- note removed: "Button Triggers"
- note removed: "I2C Pull Ups"
- note removed: "N. Seidle"
- note removed: "Power"
- note removed: "X10"
- moved on the sheet: C3, C5, C6, C7, C8, D1, J8, JP10, JP12, R10, R11, R2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
