File: Hardware/Qwiic MP3 Trigger.brd (EAGLE design)
At the start: 25.4 x 50.8 mm, 106 parts, among them J1 MICRO-SD, J2 QWIIC_RIGHT_ANGLE, J3 PTH, J4 QWIIC_RIGHT_ANGLE, J7 ISP, J8 3.5mm Audio, J9 Poke-Home, U1 TPA2005D1, U3 AP2112-3.3V, U4 ATTINY84-ARDUINO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

Commit message: Proto with MY1690
Parts:
- removed J1: MICRO-SD, SparkFun-Connectors:MICRO-SD-SOCKET
- removed U$11, U$9: (no value), Labels:INT#-[<
- removed U$13: (no value), buzzard_labels (16):#6
- removed U$16, U$7: (no value), Labels:RST#-[>
- removed U$21, U$4: (no value), Labels-0_04:3#3V2
- removed U$22, U$3: (no value), Labels-0_04:GND1
- removed U$26, U$6: (no value), Labels-0_04:SCL9
- removed U$27, U$5: (no value), Labels-0_04:SDA8
- removed U$8: (no value), Labels:I_SUPER2_C-()-03
- removed U5: WT2003SH4, SparkFun-IC-Special-Function:SO16
- added J14: MICRO-SD, SparkFun-Connectors:MICROSD-EXTERNALPIN
- added LOGO4: QWIIC_LOGO_CONNECTOR, SparkFun-Aesthetics:QWIIC_5.5MM
- added U$48: (no value), output:PHONES0
- added U$51: (no value), output:#0
- added U$52: (no value), output:TRIGGER1
- added U$53: (no value), output:#2#2
- added U$54, U$55: (no value), output:#3#1
- added U$56, U$57: (no value), output:#4#0
- added U$58: (no value), output:#GND#1
- added U$59, U$60: (no value), output:#SCL#3
- added U$61, U$62: (no value), output:#SDA#2
- added U2: MY1690-16S, MY1690:SO16
- C1: value 10uF -> 1.0uF
- C5: device SparkFun-Capacitors:0402 -> SparkFun-Capacitors:0603
- FRAME1: value FRAME-LETTER -> FRAME-LEDGER
- U$10, U$38: device buzzard_labels (16):#6 -> output:#1#3
- U$12, U$28: device buzzard_labels (16):#5 -> output:#1
- U$14: device buzzard_labels (17):SPEAKER1 -> output:#0
- U$15: device buzzard_labels (17):PHONES0 -> output:#PWR#0
- U$17: device Labels:PWR-()-03 -> output:#ADR#0
- U$18: device Labels:ADR-()-03 -> output:SPEAKER0
- U$19: device buzzard_labels (16):1_1 -> output:#GND#0
- U$2: device output:#PWR#0 -> output:TRIGGER0
- U$20: device buzzard_labels (17):SPEAKER1 -> output:#I�C#0
- U$24: device buzzard_labels (17):QWIIC_MP32 -> output:#PWR#0
- U$25: device buzzard_labels (16):#6 -> output:QWIIC_MP30
- U$29, U$45: device buzzard_labels (13):TRIGGER5 -> output:L1
- U$31: device buzzard_labels (14):43 -> output:#GND#0
- U$32: device buzzard_labels (14):21 -> output:PHONES0
- U$33: device buzzard_labels (14):32 -> output:##INT##4
- U$34: device buzzard_labels (14):43 -> output:##INT##4
- U$35: device buzzard_labels (16):GND0 -> output:##RST##5
- U$36: device buzzard_labels (14):32 -> output:##RST##5
- U$37: device buzzard_labels (16):L12 -> output:R0
- U$39: device buzzard_labels (16):R11 -> output:R0
- U$40: device buzzard_labels (17):PHONES0 -> output:SPEAKER0
- U$41: device buzzard_labels (16):L12 -> output:#2
- U$42: device buzzard_labels (14):21 -> output:#3#3V#0
- U$43: device buzzard_labels (16):R11 -> output:#2
- U$44: device buzzard_labels (16):1_1 -> output:#3#3V#0
- U$46: device buzzard_labels (16):GND0 -> output:#GND#1
- U$47: device Labels:QWIIC-LOGO-MEDIUM -> output:TRIGGER0
- U$49: device buzzard_labels (2):TRIGGER4 -> output:#2#2
- moved FRAME1 66.8 mm to (44.5, -34.3), flipped to the bottom
- moved U$46 47.8 mm to (6.35, 3.94), flipped to the top, turned to 90 degrees
- moved U$35 45.8 mm to (19.1, 3.81), turned to 90 degrees
- moved U$36 40.3 mm to (19.1, 3.81)
- moved U$34 40.1 mm to (16.5, 3.81)
- moved U$33 40.1 mm to (16.5, 3.81), flipped to the bottom
- moved U$44 39.8 mm to (8.89, 4.19), flipped to the top
- moved U$42 39.7 mm to (8.89, 4.19)
- moved U$47 29.3 mm to (6.35, 47.4), flipped to the top, turned to 90 degrees
- moved U$20 24.4 mm to (21.6, 13.3)
- moved U$2 22.1 mm to (6.48, 47.4)
- moved U$49 14.2 mm to (11.4, 45.3), flipped to the top, turned to 90 degrees
- moved U$15 12.3 mm to (22.7, 28.1), turned to 0 degrees
- moved U$25 12.2 mm to (6.86, 35.1), turned to 0 degrees
- moved U$19 11.6 mm to (19.1, 49.5), flipped to the bottom, turned to 0 degrees
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Connections:
- new net N$7: C4.1, U2.7
- net 3.3V: now also U2.12; no longer U5.11
- net 5V: now also C1.1; no longer C4.1
- net ADKEY: now also U2.4; no longer U5.7
- net D+: now also U2.6; no longer U5.5
- net D-: now also U2.5; no longer U5.4
- net GND: now also J14.10, J14.11, J14.12, J14.13, J14.6, U2.13, U2.8; no longer J1.CD1, J1.GND, U5.12, U5.8
- net MP3-RXI: now also U2.15; no longer U5.6
- net MP3-TXO: now also U2.14; no longer U5.16
- net PLAYING: now also U2.16; no longer U5.15
- net SD_CLK: now also J14.5, U2.3; no longer J1.SCLK, U5.3
- net SD_CMD: now also J14.3, U2.2; no longer J1.DI, U5.1
- net SD_DAT: now also J14.7, U2.1; no longer J1.DO, U5.2
- net VCCIO: now also J14.4, U2.11; no longer C1.1, J1.VCC, U5.10
- net VOUTL: now also U2.9; no longer U5.13
- net VOUTR: now also U2.10; no longer U5.14
Routing:
- net MP3-RXI: track 5.09 -> 23.4 mm
- net SDA: track 66.7 -> 74.0 mm
- net ADKEY: track 4.98 -> 11.9 mm
- net VCCIO: track 37.9 -> 44.1 mm
- net PLAYING: track 42.0 -> 46.8 mm, vias 2 -> 3
- net N$7: track 0.00 -> 4.00 mm, vias 0 -> 1
- net VOUTR: track 47.2 -> 43.4 mm
- net VOUTL: track 43.3 -> 39.5 mm
- net SD_DAT: track 8.49 -> 11.3 mm, vias 0 -> 2
- net MP3-TXO: track 14.1 -> 11.6 mm
- net !INT: track 38.8 -> 41.0 mm
- net D+: track 11.9 -> 13.7 mm
- net OUT-: track 16.2 -> 17.7 mm
- net !RST: track 42.2 -> 40.7 mm
- net TRIGGER1: track 47.9 -> 46.3 mm
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Other:
- board text added: "v30"
- board text removed: "v20"
